Commit message: [ros2_control_demo_robot] Add gazebo for rrbot position_only demo.

File: ros2_control_demo_robot/description/rrbot/rrbot.gazebo.xacro (robot description, xacro)
@@ -8,7 +8,6 @@
     <!-- ros_control plugin -->
     <gazebo>
-      <plugin name="gazebo_ros_control" filename="libgazebo_ros_control.so">
-        <robotNamespace>/rrbot</robotNamespace>
-        <robotSimType>gazebo_ros_control/DefaultRobotHWSim</robotSimType>
+      <plugin name="gazebo_ros2_control" filename="libgazebo_ros2_control.so">
+        <parameters>$(find ros2_control_demo_robot)/controllers/rrbot_gazebo_forward_controller_position.yaml</parameters>
       </plugin>
     </gazebo>

File: ros2_control_demo_robot/description/rrbot/rrbot_system_position_only.ros2_control.xacro (robot description, xacro)
@@ -1,12 +1,19 @@
 <?xml version="1.0"?>
 <robot xmlns:xacro="http://www.ros.org/wiki/xacro">
-  <xacro:macro name="rrbot_system_position_only" params="name prefix">
+  <xacro:macro name="rrbot_system_position_only" params="name prefix simu:='false' ">
     <ros2_control name="${name}" type="system">
-      <hardware>
-        <plugin>ros2_control_demo_hardware/RRBotSystemPositionOnlyHardware</plugin>
-        <param name="example_param_hw_start_duration_sec">2.0</param>
-        <param name="example_param_hw_stop_duration_sec">3.0</param>
-        <param name="example_param_hw_slowdown">2.0</param>
-      </hardware>
+      <xacro:if value="$(arg simu)">
+        <hardware>
+          <plugin>gazebo_ros2_control/GazeboSystem</plugin>
+        </hardware>
+      </xacro:if>
+      <xacro:unless value="$(arg simu)">
+        <hardware>
+          <plugin>ros2_control_demo_hardware/RRBotSystemPositionOnlyHardware</plugin>
+          <param name="example_param_hw_start_duration_sec">2.0</param>
+          <param name="example_param_hw_stop_duration_sec">3.0</param>
+          <param name="example_param_hw_slowdown">2.0</param>
+        </hardware>
+      </xacro:unless>
       <joint name="joint1">
         <command_interface name="position">

File: ros2_control_demo_robot/description/rrbot_system_position_only.urdf.xacro (robot description, xacro)
@@ -6,4 +6,5 @@
 -->
 <robot xmlns:xacro="http://www.ros.org/wiki/xacro" name="2dof_robot">
+  <xacro:arg name="simu" default="false" />
   <!-- Import RRBot macro -->
   <xacro:include filename="rrbot/rrbot.urdf.xacro" />
@@ -27,4 +28,4 @@
   </xacro:rrbot>
   <xacro:rrbot_gazebo prefix="" />
-  <xacro:rrbot_system_position_only name="RRBotSystemPositionOnly" prefix="" />
+  <xacro:rrbot_system_position_only name="RRBotSystemPositionOnly" prefix="" simu="$(arg simu)" />
 </robot>
