Commit message: Reorganize to new RM structure

File: ros2_control_demo_robot/description/rrbot/rrbot_system_position_only.ros2_control.xacro (robot description, xacro)
@@ -4,18 +4,22 @@
     <ros2_control name="${name}" type="system">
       <hardware>
-        <classType>ros2_control_demo_hardware/RRBotSystemPositionOnlyHardware</classType>
+        <plugin>ros2_control_demo_hardware/RRBotSystemPositionOnlyHardware</plugin>
         <param name="example_param_hw_start_duration_sec">2.0</param>
         <param name="example_param_hw_stop_duration_sec">3.0</param>
         <param name="example_param_hw_slowdown">2.0</param>
       </hardware>
-      <joint name="${prefix}joint1">
-        <classType>ros2_control_components/PositionJoint</classType>
-        <param name="min">-1</param>
-        <param name="max">1</param>
+      <joint name="joint1">
+        <command_interface name="position">
+          <param name="min">-1</param>
+          <param name="max">1</param>
+        </command_interface>
+        <state_interface name="position"/>
       </joint>
-      <joint name="${prefix}joint2">
-        <classType>ros2_control_components/PositionJoint</classType>
-        <param name="min">-1</param>
-        <param name="max">1</param>
+      <joint name="joint2">
+        <command_interface name="position">
+          <param name="min">-1</param>
+          <param name="max">1</param>
+        </command_interface>
+        <state_interface name="position"/>
       </joint>
     </ros2_control>

File: ros2_control_demo_robot/description/rrbot_system_position_only.urdf.xacro (robot description, xacro)
@@ -27,4 +27,4 @@
   </xacro:rrbot>
   <xacro:rrbot_gazebo prefix="" />
-  <xacro:rrbot_system_position_only name="RRBot_System_Position_Only" prefix="" />
+  <xacro:rrbot_system_position_only name="RRBotSystemPositionOnly" prefix="" />
 </robot>

Commit message: [ros2_control_demo_robot] Change xacro parameter simu to use_simu

File: ros2_control_demo_robot/description/rrbot/rrbot_system_position_only.ros2_control.xacro (robot description, xacro)
@@ -1,12 +1,12 @@
 <?xml version="1.0"?>
 <robot xmlns:xacro="http://www.ros.org/wiki/xacro">
-  <xacro:macro name="rrbot_system_position_only" params="name prefix simu:='false' ">
+  <xacro:macro name="rrbot_system_position_only" params="name prefix use_sim:='false' ">
     <ros2_control name="${name}" type="system">
-      <xacro:if value="$(arg simu)">
+      <xacro:if value="$(arg use_sim)">
         <hardware>
           <plugin>gazebo_ros2_control/GazeboSystem</plugin>
         </hardware>
       </xacro:if>
-      <xacro:unless value="$(arg simu)">
+      <xacro:unless value="$(arg use_sim)">
         <hardware>
           <plugin>ros2_control_demo_hardware/RRBotSystemPositionOnlyHardware</plugin>

File: ros2_control_demo_robot/description/rrbot_system_position_only.urdf.xacro (robot description, xacro)
@@ -6,5 +6,5 @@
 -->
 <robot xmlns:xacro="http://www.ros.org/wiki/xacro" name="2dof_robot">
-  <xacro:arg name="simu" default="false" />
+  <xacro:arg name="use_sim" default="false" />
   <!-- Import RRBot macro -->
   <xacro:include filename="rrbot/rrbot.urdf.xacro" />
@@ -28,4 +28,4 @@
   </xacro:rrbot>
   <xacro:rrbot_gazebo prefix="" />
-  <xacro:rrbot_system_position_only name="RRBotSystemPositionOnly" prefix="" simu="$(arg simu)" />
+  <xacro:rrbot_system_position_only name="RRBotSystemPositionOnly" prefix="" use_sim="$(arg use_sim)" />
 </robot>
