Commit message: Adjust colors of the robot

File: ros2_control_demo_robot/description/rrbot/rrbot.materials.xacro (robot description, xacro)
@@ -26,4 +26,7 @@
     <color rgba="0.8 0.0 0.0 1.0"/>
   </material>
+  <material name="yellow">
+    <color rgba="1.0 1.0 0.0 1.0"/>
+  </material>
   <material name="white">
     <color rgba="1.0 1.0 1.0 1.0"/>

File: ros2_control_demo_robot/description/rrbot/rrbot.urdf.xacro (robot description, xacro)
@@ -28,5 +28,5 @@
         <box size="${width} ${width} ${height1}"/>
       </geometry>
-      <material name="brown"/>
+      <material name="orange"/>
     </visual>
     <inertial>
@@ -59,5 +59,5 @@
           <box size="${width} ${width} ${height2}"/>
         </geometry>
-        <material name="blue"/>
+        <material name="yellow"/>
       </visual>
       <inertial>
