Commit message: Final chnages of test nodes and added JTC for demo HW

File: ros2_control_demo_robot/description/rrbot/rrbot.urdf.xacro (robot description, xacro)
@@ -3,8 +3,7 @@
   <xacro:macro name="rrbot" params="parent prefix *origin">
   <!-- Constants for robot dimensions -->
-  <xacro:property name="PI" value="3.1415926535897931"/>
   <xacro:property name="mass" value="1" /> <!-- arbitrary value for mass -->
   <xacro:property name="width" value="0.1" /> <!-- Square dimensions (widthxwidth) of beams -->
-  <xacro:property name="height1" value="2" /> <!-- Link 1 -->
+  <xacro:property name="height1" value="0.2" /> <!-- Link 1 -->
   <xacro:property name="height2" value="1" /> <!-- Link 2 -->
   <xacro:property name="height3" value="1" /> <!-- Link 3 -->
@@ -29,5 +28,5 @@
         <box size="${width} ${width} ${height1}"/>
       </geometry>
-      <material name="orange"/>
+      <material name="brown"/>
     </visual>
     <inertial>
@@ -60,5 +59,5 @@
           <box size="${width} ${width} ${height2}"/>
         </geometry>
-        <material name="black"/>
+        <material name="blue"/>
       </visual>
       <inertial>

File: ros2_control_demo_robot/description/rrbot/rrbot_system_position_only.ros2_control.xacro (robot description, xacro)
@@ -1,5 +1,5 @@
 <?xml version="1.0"?>
 <robot xmlns:xacro="http://www.ros.org/wiki/xacro">
-  <xacro:macro name="rrbot_system_position_only" params="name prefix">
+  <xacro:macro name="rrbot_system_position_only" params="name prefix slowdown:=2.0">
     <ros2_control name="${name}" type="system">
       <hardware>
@@ -7,5 +7,5 @@
         <param name="example_param_hw_start_duration_sec">2.0</param>
         <param name="example_param_hw_stop_duration_sec">3.0</param>
-        <param name="example_param_hw_slowdown">2.0</param>
+        <param name="example_param_hw_slowdown">${slowdown}</param>
       </hardware>
       <joint name="joint1">

File: ros2_control_demo_robot/description/rrbot_system_position_only.urdf.xacro (robot description, xacro)
@@ -6,16 +6,14 @@
 -->
 <robot xmlns:xacro="http://www.ros.org/wiki/xacro" name="2dof_robot">
+  <!-- Enable setting arguments from the launch file -->
+  <xacro:arg name="slowdown" default="2.0" />
   <!-- Import RRBot macro -->
-  <xacro:include filename="rrbot/rrbot.urdf.xacro" />
-  <!-- <xacro:include filename="$(find ros2_control_demo_robot)/description/rrbot/rrbot.urdf.xacro" /> -->
+  <xacro:include filename="$(find ros2_control_demo_robot)/description/rrbot/rrbot.urdf.xacro" />
   <!-- Import all Gazebo-customization elements, including Gazebo colors -->
-  <xacro:include filename="rrbot/rrbot.gazebo.xacro" />
-  <!-- <xacro:include filename="$(find ros2_control_demo_robot)/description/rrbot/rrbot.gazebo.xacro" /> -->
+  <xacro:include filename="$(find ros2_control_demo_robot)/description/rrbot/rrbot.gazebo.xacro" />
   <!-- Import Rviz colors -->
-  <xacro:include filename="rrbot/rrbot.materials.xacro" />
-  <!-- <xacro:include filename="$(find ros2_control_demo_robot)/description/rrbot/rrbot.materials.xacro" /> -->
+  <xacro:include filename="$(find ros2_control_demo_robot)/description/rrbot/rrbot.materials.xacro" />
   <!-- Import RRBot ros2_control description -->
-  <xacro:include filename="rrbot/rrbot_system_position_only.ros2_control.xacro" />
-  <!-- <xacro:include filename="$(find ros2_control_demo_robot)/description/rrbot/rrbot_system_position_only.ros2_control.xacro" /> -->
+  <xacro:include filename="$(find ros2_control_demo_robot)/description/rrbot/rrbot_system_position_only.ros2_control.xacro" />
   <!-- Used for fixing robot -->
   <link name="world"/>
@@ -27,4 +25,4 @@
   </xacro:rrbot>
   <xacro:rrbot_gazebo prefix="" />
-  <xacro:rrbot_system_position_only name="RRBotSystemPositionOnly" prefix="" />
+  <xacro:rrbot_system_position_only name="RRBotSystemPositionOnly" prefix="" slowdown="$(arg slowdown)" />
 </robot>

Commit message: Add corrections and extensions for the rrbot

File: ros2_control_demo_robot/description/rrbot/rrbot.urdf.xacro (robot description, xacro)
@@ -28,5 +28,5 @@
         <box size="${width} ${width} ${height1}"/>
       </geometry>
-      <material name="orange"/>
+      <material name="brown"/>
     </visual>
     <inertial>

Commit message: Adjust colors of the robot

File: ros2_control_demo_robot/description/rrbot/rrbot.urdf.xacro (robot description, xacro)
@@ -28,5 +28,5 @@
         <box size="${width} ${width} ${height1}"/>
       </geometry>
-      <material name="brown"/>
+      <material name="orange"/>
     </visual>
     <inertial>

Commit message: Add corrections and extensions for the rrbot (#71)
* Add corrections and extensions for the rrbot

* Correct build and remove demo nodes from readme.

* Apply suggestions from code review

Co-authored-by: Bence Magyar <bence.magyar.robotics@gmail.com>

* Adjust colors of the robot

* Update ros2_control_demo_robot/package.xml

Co-authored-by: Victor Lopez <3469405+v-lopez@users.noreply.github.com>

* Update ros2_control_demo_robot/launch/test_rrbot_description.launch.py

Co-authored-by: Bence Magyar <bence.magyar.robotics@gmail.com>
Co-authored-by: Victor Lopez <3469405+v-lopez@users.noreply.github.com>

File: ros2_control_demo_robot/description/rrbot/rrbot.urdf.xacro (robot description, xacro)
@@ -3,8 +3,7 @@
   <xacro:macro name="rrbot" params="parent prefix *origin">
   <!-- Constants for robot dimensions -->
-  <xacro:property name="PI" value="3.1415926535897931"/>
   <xacro:property name="mass" value="1" /> <!-- arbitrary value for mass -->
   <xacro:property name="width" value="0.1" /> <!-- Square dimensions (widthxwidth) of beams -->
-  <xacro:property name="height1" value="2" /> <!-- Link 1 -->
+  <xacro:property name="height1" value="0.2" /> <!-- Link 1 -->
   <xacro:property name="height2" value="1" /> <!-- Link 2 -->
   <xacro:property name="height3" value="1" /> <!-- Link 3 -->
@@ -60,5 +59,5 @@
           <box size="${width} ${width} ${height2}"/>
         </geometry>
-        <material name="black"/>
+        <material name="yellow"/>
       </visual>
       <inertial>
