Commit message: Adding changes for SR_issue_2

File: ros2_control_demo_robot/description/rrbot/rrbot_system_with_sensor.ros2_control.xacro (robot description, xacro)
@@ -1,12 +1,20 @@
 <?xml version="1.0"?>
 <robot xmlns:xacro="http://www.ros.org/wiki/xacro">
-  <xacro:macro name="rrbot_system_with_sensor" params="name prefix slowdown:=2.0">
+  <xacro:macro name="rrbot_system_with_sensor" params="name prefix
+  use_fake_hardware:=^|true fake_sensor_commands:=^|false slowdown:=2.0">
     <ros2_control name="${name}" type="system">
       <hardware>
-        <plugin>ros2_control_demo_hardware/RRBotSystemWithSensorHardware</plugin>
-        <param name="example_param_hw_start_duration_sec">2.0</param>
-        <param name="example_param_hw_stop_duration_sec">3.0</param>
-        <param name="example_param_hw_slowdown">${slowdown}</param>
-        <param name="example_param_max_sensor_change">5.0</param>
+        <xacro:if value="${use_fake_hardware}">
+          <plugin>fake_components/GenericSystem</plugin>
+          <param name="fake_sensor_commands">${fake_sensor_commands}</param>
+          <param name="state_following_offset">0.0</param>
+        </xacro:if>
+        <xacro:unless value="${use_fake_hardware}">
+          <plugin>ros2_control_demo_hardware/RRBotSystemWithSensorHardware</plugin>
+          <param name="example_param_hw_start_duration_sec">2.0</param>
+          <param name="example_param_hw_stop_duration_sec">3.0</param>
+          <param name="example_param_hw_slowdown">${slowdown}</param>
+          <param name="example_param_max_sensor_change">5.0</param>
+        </xacro:unless>
       </hardware>
       <joint name="joint1">

File: ros2_control_demo_robot/description/rrbot_system_with_sensor.urdf.xacro (robot description, xacro)
@@ -2,9 +2,12 @@
 <!-- Revolute-Revolute Manipulator with a 2D Force-Torque sensor -->
 <!--
-Copied and modified from ROS1 example:
+Copied and modified from ROS1 example -
 https://github.com/ros-simulation/gazebo_ros_demos/blob/kinetic-devel/rrbot_description/urdf/rrbot.xacro
 -->
 <robot xmlns:xacro="http://www.ros.org/wiki/xacro" name="2dof_robot">
   <!-- Enable setting arguments from the launch file -->
+  <xacro:arg name="use_fake_hardware" default="true" />
+  <xacro:arg name="fake_sensor_commands" default="false" />
+  <xacro:arg name="prefix" default="" />
   <xacro:arg name="slowdown" default="2.0" />
   <!-- Import RRBot macro -->
@@ -21,8 +24,12 @@
     <static>true</static>
   </gazebo>
-  <xacro:rrbot parent="world" prefix="">
+  <xacro:rrbot parent="world" prefix="$(arg prefix)">
     <origin xyz="0 0 0" rpy="0 0 0" />
   </xacro:rrbot>
   <xacro:rrbot_gazebo prefix="" />
-  <xacro:rrbot_system_with_sensor name="RRBotSystemWithSensor" prefix="" />
+  <xacro:rrbot_system_with_sensor
+    name="RRBotSystemWithSensor" prefix="$(arg prefix)"
+    use_fake_hardware="$(arg use_fake_hardware)"
+    fake_sensor_commands="$(arg fake_sensor_commands)"
+    slowdown="$(arg slowdown)" />
 </robot>

Commit message: Example-3 : Adapting changes from PR-76

File: ros2_control_demo_robot/description/rrbot/rrbot_system_with_sensor.ros2_control.xacro (robot description, xacro)
@@ -1,21 +1,27 @@
 <?xml version="1.0"?>
 <robot xmlns:xacro="http://www.ros.org/wiki/xacro">
-  <xacro:macro name="rrbot_system_with_sensor" params="name prefix
-  use_fake_hardware:=^|true fake_sensor_commands:=^|false slowdown:=2.0">
+  <xacro:macro name="rrbot_system_with_sensor" params="name prefix use_sim:=^|false use_fake_hardware:=^|true fake_sensor_commands:=^|false slowdown:=2.0">
     <ros2_control name="${name}" type="system">
-      <hardware>
-        <xacro:if value="${use_fake_hardware}">
-          <plugin>fake_components/GenericSystem</plugin>
-          <param name="fake_sensor_commands">${fake_sensor_commands}</param>
-          <param name="state_following_offset">0.0</param>
-        </xacro:if>
-        <xacro:unless value="${use_fake_hardware}">
-          <plugin>ros2_control_demo_hardware/RRBotSystemWithSensorHardware</plugin>
-          <param name="example_param_hw_start_duration_sec">2.0</param>
-          <param name="example_param_hw_stop_duration_sec">3.0</param>
-          <param name="example_param_hw_slowdown">${slowdown}</param>
-          <param name="example_param_max_sensor_change">5.0</param>
-        </xacro:unless>
-      </hardware>
+      <xacro:if value="$(arg use_sim)">
+        <hardware>
+          <plugin>gazebo_ros2_control/GazeboSystem</plugin>
+        </hardware>
+      </xacro:if>
+      <xacro:unless value="$(arg use_sim)">
+        <hardware>
+          <xacro:if value="${use_fake_hardware}">
+            <plugin>fake_components/GenericSystem</plugin>
+            <param name="fake_sensor_commands">${fake_sensor_commands}</param>
+            <param name="state_following_offset">0.0</param>
+          </xacro:if>
+          <xacro:unless value="${use_fake_hardware}">
+            <plugin>ros2_control_demo_hardware/RRBotSystemWithSensorHardware</plugin>
+            <param name="example_param_hw_start_duration_sec">2.0</param>
+            <param name="example_param_hw_stop_duration_sec">3.0</param>
+            <param name="example_param_hw_slowdown">${slowdown}</param>
+            <param name="example_param_max_sensor_change">5.0</param>
+          </xacro:unless>
+        </hardware>
+      </xacro:unless>
       <joint name="joint1">
         <command_interface name="position">
@@ -33,6 +39,10 @@
       </joint>
       <sensor name="tcp_fts_sensor">
-        <state_interface name="fx"/>
-        <state_interface name="tz"/>
+        <state_interface name="mysensor_force.x"/>
+        <state_interface name="mysensor_force.y"/>
+        <state_interface name="mysensor_force.z"/>
+        <state_interface name="mysensor_torque.x"/>
+        <state_interface name="mysensor_torque.y"/>
+        <state_interface name="mysensor_torque.z"/>
         <param name="frame_id">rrbot_tcp</param>
         <param name="fx_range">100</param>

File: ros2_control_demo_robot/description/rrbot_system_with_sensor.urdf.xacro (robot description, xacro)
@@ -12,11 +12,11 @@
   <xacro:arg name="slowdown" default="2.0" />
   <!-- Import RRBot macro -->
-  <xacro:include filename="$(find ros2_control_demo_robot)/description/rrbot/rrbot.urdf.xacro" />
+  <xacro:include filename="$(find ros2_control_demo_description)/urdf/rrbot/rrbot.urdf.xacro" />
   <!-- Import all Gazebo-customization elements, including Gazebo colors -->
-  <xacro:include filename="$(find ros2_control_demo_robot)/description/rrbot/rrbot.gazebo.xacro" />
+  <xacro:include filename="$(find ros2_control_demo_description)/urdf/rrbot/gazebo/rrbot.gazebo.xacro" />
   <!-- Import Rviz colors -->
-  <xacro:include filename="$(find ros2_control_demo_robot)/description/rrbot/rrbot.materials.xacro" />
+  <xacro:include filename="$(find ros2_control_demo_description)/urdf/rrbot/gazebo/rrbot.materials.xacro" />
   <!-- Import RRBot ros2_control description -->
-  <xacro:include filename="$(find ros2_control_demo_robot)/description/rrbot/rrbot_system_with_sensor.ros2_control.xacro" />
+  <xacro:include filename="$(find ros2_control_demo_description)/urdf/rrbot/ros2_control/rrbot_system_with_sensor.ros2_control.xacro" />
   <!-- Used for fixing robot -->
   <link name="world"/>
@@ -27,5 +27,5 @@
     <origin xyz="0 0 0" rpy="0 0 0" />
   </xacro:rrbot>
-  <xacro:rrbot_gazebo prefix="" />
+  <xacro:rrbot_gazebo prefix="$(arg prefix)" />
   <xacro:rrbot_system_with_sensor
     name="RRBotSystemWithSensor" prefix="$(arg prefix)"
