Commit message: applying review suggestions

File: ros2_control_demo_robot/description/diffbot/diffbot.urdf.xacro (robot description, xacro)
@@ -1,5 +1,5 @@
 <?xml version="1.0"?>
 <robot xmlns:xacro="http://www.ros.org/wiki/xacro">
-  <xacro:macro name="diffbot" params="parent prefix *origin">
+  <xacro:macro name="diffbot" params="prefix">
   <!-- Constants for robot dimensions -->
   <xacro:property name="PI" value="3.1415926535897931"/>
@@ -11,10 +11,7 @@
   <xacro:property name="wheel_len" value="0.020" />
   <xacro:property name="wheel_radius" value="0.015" />
+  <xacro:property name="caster_wheel_mass" value="0.1" /> <!-- arbitrary value for caster wheel mass -->
+  <xacro:property name="caster_wheel_radius" value="0.015" />
   <xacro:property name="z_offset" value="-${base_height/2}" /> <!-- Space btw top of beam and the each joint -->
-  <joint name="${prefix}base_joint" type="fixed">
-    <xacro:insert_block name="origin" />
-    <parent link="${parent}"/>
-    <child link="${prefix}base_link" />
-  </joint>
   <!-- Base Link -->
   <link name="${prefix}base_link">
@@ -103,4 +100,62 @@
         </inertial>
       </link>
+    <joint name="${prefix}caster_frontal_wheel_joint" type="fixed">
+      <parent link="${prefix}base_link"/>
+      <child link="${prefix}caster_frontal_wheel"/>
+      <origin xyz="${base_width/2 - caster_wheel_radius} 0 ${z_offset}" rpy="0 0 0"/>
+    </joint>
+    <!-- caster frontal wheel Link -->
+    <link name="${prefix}caster_frontal_wheel">
+      <collision>
+        <origin xyz="0 0 0" rpy="0 0 0"/>
+        <geometry>
+          <sphere radius="${caster_wheel_radius}"/>
+        </geometry>
+      </collision>
+      <visual>
+        <origin xyz="0 0 0" rpy="0 0 0"/>
+        <geometry>
+          <sphere radius="${caster_wheel_radius}"/>
+        </geometry>
+        <material name="white"/>
+      </visual>
+      <inertial>
+        <origin xyz="0 0 0" rpy="0 0 0"/>
+        <mass value="${caster_wheel_mass}"/>
+        <inertia
+          ixx="${caster_wheel_mass * 0.4 * (caster_wheel_radius * caster_wheel_radius)}" ixy="0.0" ixz="0.0"
+          iyy="${caster_wheel_mass * 0.4 * (caster_wheel_radius * caster_wheel_radius)}" iyz="0.0"
+          izz="${caster_wheel_mass * 0.4 * (caster_wheel_radius * caster_wheel_radius)}"/>
+        </inertial>
+      </link>
+    <joint name="${prefix}caster_rear_wheel_joint" type="fixed">
+      <parent link="${prefix}base_link"/>
+      <child link="${prefix}caster_rear_wheel"/>
+      <origin xyz="${-base_width/2 + caster_wheel_radius} 0 ${z_offset}" rpy="0 0 0"/>
+    </joint>
+    <!-- caster rear wheel Link -->
+    <link name="${prefix}caster_rear_wheel">
+      <collision>
+        <origin xyz="0 0 0" rpy="0 0 0"/>
+        <geometry>
+          <sphere radius="${caster_wheel_radius}"/>
+        </geometry>
+      </collision>
+      <visual>
+        <origin xyz="0 0 0" rpy="0 0 0"/>
+        <geometry>
+          <sphere radius="${caster_wheel_radius}"/>
+        </geometry>
+        <material name="white"/>
+      </visual>
+      <inertial>
+        <origin xyz="0 0 0" rpy="0 0 0"/>
+        <mass value="${caster_wheel_mass}"/>
+        <inertia
+          ixx="${caster_wheel_mass * 0.4 * (caster_wheel_radius * caster_wheel_radius)}" ixy="0.0" ixz="0.0"
+          iyy="${caster_wheel_mass * 0.4 * (caster_wheel_radius * caster_wheel_radius)}" iyz="0.0"
+          izz="${caster_wheel_mass * 0.4 * (caster_wheel_radius * caster_wheel_radius)}"/>
+        </inertial>
+      </link>
   </xacro:macro>
 </robot>

File: ros2_control_demo_robot/description/diffbot/diffbot_system.ros2_control.xacro (robot description, xacro)
@@ -10,40 +10,20 @@
       </hardware>
       <joint name="left_wheel_joint">
-        <state_interface name="position"/>
         <command_interface name="velocity">
           <param name="min">-1</param>
           <param name="max">1</param>
         </command_interface>
+        <state_interface name="position"/>
         <state_interface name="velocity"/>
       </joint>
       <joint name="right_wheel_joint">
-        <state_interface name="position"/>
         <command_interface name="velocity">
           <param name="min">-1</param>
           <param name="max">1</param>
         </command_interface>
+        <state_interface name="position"/>
         <state_interface name="velocity"/>
       </joint>
     </ros2_control>
-  <!-- <ros2_control name="TestActuatorHardwareLeft" type="actuator">
-    <hardware>
-      <plugin>test_actuator</plugin>
-    </hardware>
-    <joint name="left_wheel_joint">
-      <state_interface name="position"/>
-      <command_interface name="velocity"/>
-      <state_interface name="velocity"/>
-    </joint>
-  </ros2_control>
-  <ros2_control name="TestActuatorHardwareRight" type="actuator">
-    <hardware>
-      <plugin>test_actuator</plugin>
-    </hardware>
-    <joint name="right_wheel_joint">
-      <state_interface name="position"/>
-      <command_interface name="velocity"/>
-      <state_interface name="velocity"/>
-    </joint>
-  </ros2_control> -->
   </xacro:macro>
 </robot>

File: ros2_control_demo_robot/description/diffbot_system.urdf.xacro (robot description, xacro)
@@ -6,5 +6,4 @@
 -->
 <robot xmlns:xacro="http://www.ros.org/wiki/xacro" name="2dof_robot">
-  <!-- Import diffbot macro -->
   <xacro:include filename="diffbot/diffbot.urdf.xacro" />
   <!-- <xacro:include filename="$(find ros2_control_demo_robot)/description/diffbot/diffbot.urdf.xacro" /> -->
@@ -18,12 +17,5 @@
   <xacro:include filename="diffbot/diffbot_system.ros2_control.xacro" />
   <!-- <xacro:include filename="$(find ros2_control_demo_robot)/description/diffbot/diffbot_system.ros2_control.xacro" /> -->
-  <!-- Used for fixing robot -->
-  <link name="world"/>
-  <gazebo reference="world">
-    <static>true</static>
-  </gazebo>
-  <xacro:diffbot parent="world" prefix="">
-    <origin xyz="0 0 0" rpy="0 0 0" />
-  </xacro:diffbot>
+  <xacro:diffbot prefix="" />
   <xacro:diffbot_gazebo prefix="" />
   <xacro:diffbot_system name="DiffBotSystem" prefix="" />
