Commit message: applying review suggestions

File: ros2_control_demo_robot/description/diffbot/diffbot.gazebo.xacro (robot description, xacro)
@@ -6,14 +6,7 @@
 <robot xmlns:xacro="http://ros.org/wiki/xacro">
   <xacro:macro name="diffbot_gazebo" params="prefix">
-    <!-- ros_control plugin -->
-    <gazebo>
-      <plugin name="gazebo_ros_control" filename="libgazebo_ros_control.so">
-        <robotNamespace>/diffbot</robotNamespace>
-        <robotSimType>gazebo_ros_control/DefaultRobotHWSim</robotSimType>
-      </plugin>
-    </gazebo>
     <!-- Link1 -->
     <gazebo reference="${prefix}base_link">
-      <material>Gazebo/Orange</material>
+      <material>Gazebo/Blue</material>
     </gazebo>
     <!-- Link2 -->
@@ -27,5 +20,5 @@
       <mu1>0.2</mu1>
       <mu2>0.2</mu2>
-      <material>Gazebo/Orange</material>
+      <material>Gazebo/Black</material>
     </gazebo>
     <!-- camera_link -->
@@ -34,40 +27,4 @@
       <mu2>0.2</mu2>
       <material>Gazebo/Red</material>
-    </gazebo>
-    <!-- hokuyo -->
-    <gazebo reference="${prefix}hokuyo_link">
-      <sensor type="gpu_ray" name="head_hokuyo_sensor">
-        <pose>0 0 0 0 0 0</pose>
-        <visualize>false</visualize>
-        <update_rate>40</update_rate>
-        <ray>
-          <scan>
-            <horizontal>
-              <samples>720</samples>
-              <resolution>1</resolution>
-              <min_angle>-1.570796</min_angle>
-              <max_angle>1.570796</max_angle>
-            </horizontal>
-          </scan>
-          <range>
-            <min>0.10</min>
-            <max>30.0</max>
-            <resolution>0.01</resolution>
-          </range>
-          <noise>
-            <type>gaussian</type>
-            <!-- Noise parameters based on published spec for Hokuyo laser
-            achieving "+-30mm" accuracy at range < 10m.  A mean of 0.0m and
-            stddev of 0.01m will put 99.7% of samples within 0.03m of the true
-            reading. -->
-            <mean>0.0</mean>
-            <stddev>0.01</stddev>
-          </noise>
-        </ray>
-        <plugin name="gazebo_ros_head_hokuyo_controller" filename="libgazebo_ros_gpu_laser.so">
-          <topicName>/diffbot/laser/scan</topicName>
-          <frameName>hokuyo_link</frameName>
-        </plugin>
-      </sensor>
     </gazebo>
     <!-- camera -->

File: ros2_control_demo_robot/description/diffbot_system.urdf.xacro (robot description, xacro)
@@ -1,4 +1,4 @@
 <?xml version="1.0"?>
-<!-- Revolute-Revolute Manipulator -->
+<!-- Basic differential drive mobile base -->
 <!--
 Copied and modified from ROS1 example:
