Commit message: Add correction to rrbot launch using arguments and reuse the main file for starting examples.

File: ros2_control_demo_robot/description/diffbot/diffbot_system.ros2_control.xacro (robot description, xacro)
@@ -1,10 +1,17 @@
 <?xml version="1.0"?>
 <robot xmlns:xacro="http://www.ros.org/wiki/xacro">
-  <xacro:macro name="diffbot_system" params="name prefix">
+  <xacro:macro name="rrbot_system_position_only" params="name prefix use_fake_hardware:=^|true fake_sensor_commands:=^|false slowdown:=2.0">
     <ros2_control name="${name}" type="system">
       <hardware>
-        <plugin>ros2_control_demo_hardware/DiffBotSystemHardware</plugin>
-        <param name="example_param_hw_start_duration_sec">2.0</param>
-        <param name="example_param_hw_stop_duration_sec">3.0</param>
+        <xacro:if value="${use_fake_hardware}">
+          <plugin>fake_components/GenericSystem</plugin>
+          <param name="fake_sensor_commands">${fake_sensor_commands}</param>
+          <param name="state_following_offset">0.0</param>
+        </xacro:if>
+        <xacro:unless value="${use_fake_hardware}">
+          <plugin>ros2_control_demo_hardware/DiffBotSystemHardware</plugin>
+          <param name="example_param_hw_start_duration_sec">2.0</param>
+          <param name="example_param_hw_stop_duration_sec">3.0</param>
+        </xacro:unless>
       </hardware>
       <joint name="left_wheel_joint">

File: ros2_control_demo_robot/description/rrbot/gazebo/rrbot.gazebo.xacro (robot description, xacro)
@@ -1,5 +1,5 @@
 <?xml version="1.0"?>
 <!--
-Copied and modified from ROS1 example:
+Copied and modified from ROS1 example -
 https://github.com/ros-simulation/gazebo_ros_demos/blob/kinetic-devel/rrbot_description/urdf/rrbot.gazebo
 -->

File: ros2_control_demo_robot/description/rrbot/gazebo/rrbot.materials.xacro (robot description, xacro)
@@ -1,5 +1,5 @@
 <?xml version="1.0"?>
 <!--
-Copied from ROS1 example:
+Copied from ROS1 example -
 https://github.com/ros-simulation/gazebo_ros_demos/blob/kinetic-devel/rrbot_description/urdf/materials.xacro
 -->

File: ros2_control_demo_robot/description/rrbot/rrbot_system_position_only.urdf.xacro (robot description, xacro)
@@ -2,5 +2,5 @@
 <!-- Revolute-Revolute Manipulator -->
 <!--
-Copied and modified from ROS1 example:
+Copied and modified from ROS1 example -
 https://github.com/ros-simulation/gazebo_ros_demos/blob/kinetic-devel/rrbot_description/urdf/rrbot.xacro
 -->
@@ -8,4 +8,7 @@
   <xacro:arg name="use_sim" default="false" />
   <!-- Enable setting arguments from the launch file -->
+  <xacro:arg name="use_fake_hardware" default="true" />
+  <xacro:arg name="fake_sensor_commands" default="false" />
+  <xacro:arg name="prefix" default="" />
   <xacro:arg name="slowdown" default="2.0" />
   <!-- Import RRBot macro -->
@@ -22,8 +25,12 @@
     <static>true</static>
   </gazebo>
-  <xacro:rrbot parent="world" prefix="">
+  <xacro:rrbot parent="world" prefix="$(arg prefix)">
     <origin xyz="0 0 0" rpy="0 0 0" />
   </xacro:rrbot>
-  <xacro:rrbot_gazebo prefix="" />
-  <xacro:rrbot_system_position_only name="RRBotSystemPositionOnly" prefix="" use_sim="$(arg use_sim)" slowdown="$(arg slowdown)" />
+  <xacro:rrbot_gazebo prefix="$(arg prefix)" />
+  <xacro:rrbot_system_position_only
+    name="RRBotSystemPositionOnly" prefix="$(arg prefix)"
+    use_fake_hardware="$(arg use_fake_hardware)"
+    fake_sensor_commands="$(arg fake_sensor_commands)"
+    slowdown="$(arg slowdown)" />
 </robot>
