Commit message: organize urdf files to work with gazebo
Signed-off-by: Karsten Knese <Karsten1987@users.noreply.github.com>

File: ros2_control_demo_robot/description/rrbot/gazebo/rrbot.gazebo.xacro (robot description, xacro)
@@ -9,5 +9,5 @@
     <gazebo>
       <plugin name="gazebo_ros2_control" filename="libgazebo_ros2_control.so">
-        <parameters>$(find ros2_control_demo_robot)/controllers/rrbot_gazebo_forward_controller_position.yaml</parameters>
+        <parameters>$(find ros2_control_demo_robot)/config/rrbot_gazebo_forward_controller_position.yaml</parameters>
       </plugin>
     </gazebo>
@@ -64,5 +64,5 @@
           </noise>
         </ray>
-        <plugin name="gazebo_ros_head_hokuyo_controller" filename="libgazebo_ros_gpu_laser.so">
+        <plugin name="gazebo_ros_head_hokuyo_controller" filename="libgazebo_ros_ray_sensor.so">
           <topicName>/rrbot/laser/scan</topicName>
           <frameName>hokuyo_link</frameName>

File: ros2_control_demo_robot/description/rrbot/rrbot_system_position_only.urdf.xacro (robot description, xacro)
@@ -10,11 +10,11 @@
   <xacro:arg name="slowdown" default="2.0" />
   <!-- Import RRBot macro -->
-  <xacro:include filename="$(find ros2_control_demo_robot)/description/rrbot/rrbot.urdf.xacro" />
+  <xacro:include filename="$(find ros2_control_demo_robot)/description/rrbot/urdf/rrbot.urdf.xacro" />
   <!-- Import all Gazebo-customization elements, including Gazebo colors -->
-  <xacro:include filename="$(find ros2_control_demo_robot)/description/rrbot/rrbot.gazebo.xacro" />
+  <xacro:include filename="$(find ros2_control_demo_robot)/description/rrbot/gazebo/rrbot.gazebo.xacro" />
   <!-- Import Rviz colors -->
-  <xacro:include filename="$(find ros2_control_demo_robot)/description/rrbot/rrbot.materials.xacro" />
+  <xacro:include filename="$(find ros2_control_demo_robot)/description/rrbot/gazebo/rrbot.materials.xacro" />
   <!-- Import RRBot ros2_control description -->
-  <xacro:include filename="$(find ros2_control_demo_robot)/description/rrbot/rrbot_system_position_only.ros2_control.xacro" />
+  <xacro:include filename="$(find ros2_control_demo_robot)/description/rrbot/ros2_control/rrbot_system_position_only.ros2_control.xacro" />
   <!-- Used for fixing robot -->
   <link name="world"/>

File: ros2_control_demo_robot/description/rrbot/urdf/rrbot.urdf.xacro (robot description, xacro)
@@ -126,5 +126,7 @@
             <origin xyz="0 0 0" rpy="0 0 0"/>
             <geometry>
-              <mesh filename="package://rrbot_description/meshes/hokuyo.dae"/>
+              <mesh filename="package://ros2_control_demo_robot/description/rrbot/meshes/hokuyo.dae"/>
+              <!-- use model:// when downloading from the gazebo model database -->
+              <!-- <mesh filename="model://hokuyo"/> -->
             </geometry>
           </visual>
