Commit message: Move all files

File: ros2_control_demo_description/urdf/rrbot/ros2_control/rrbot_system_multi_interface.ros2_control.xacro (robot description, xacro)
@@ -1,12 +1,26 @@
 <?xml version="1.0"?>
 <robot xmlns:xacro="http://www.ros.org/wiki/xacro">
-  <xacro:macro name="rrbot_system_multi_interface" params="name prefix">
+  <xacro:macro name="rrbot_system_multi_interface" params="name prefix use_sim:=^|false use_fake_hardware:=^|true fake_sensor_commands:=^|false slowdown:=2.0">
     <ros2_control name="${name}" type="system">
-      <hardware>
-        <plugin>ros2_control_demo_hardware/RRBotSystemMultiInterfaceHardware</plugin>
-        <param name="example_param_hw_start_duration_sec">2.0</param>
-        <param name="example_param_hw_stop_duration_sec">3.0</param>
-        <param name="example_param_hw_slowdown">2.0</param>
-      </hardware>
+      <xacro:if value="$(arg use_sim)">
+        <hardware>
+          <plugin>gazebo_ros2_control/GazeboSystem</plugin>
+        </hardware>
+      </xacro:if>
+      <xacro:unless value="$(arg use_sim)">
+        <hardware>
+          <xacro:if value="${use_fake_hardware}">
+            <plugin>fake_components/GenericSystem</plugin>
+            <param name="fake_sensor_commands">${fake_sensor_commands}</param>
+            <param name="state_following_offset">0.0</param>
+          </xacro:if>
+          <xacro:unless value="${use_fake_hardware}">
+            <plugin>ros2_control_demo_hardware/RRBotSystemMultiInterfaceHardware</plugin>
+            <param name="example_param_hw_start_duration_sec">2.0</param>
+            <param name="example_param_hw_stop_duration_sec">3.0</param>
+            <param name="example_param_hw_slowdown">${slowdown}</param>
+          </xacro:unless>
+        </hardware>
+      </xacro:unless>
       <joint name="joint1">
         <command_interface name="position">
