Commit message: Update readme and test rrbot examples.

File: ros2_control_demo_description/urdf/rrbot/rrbot.urdf.xacro (robot description, xacro)
@@ -126,5 +126,5 @@
             <origin xyz="0 0 0" rpy="0 0 0"/>
             <geometry>
-              <mesh filename="package://rrbot_description/meshes/hokuyo.dae"/>
+              <mesh filename="package://ros2_control_demo_description/meshes/hokuyo.dae"/>
             </geometry>
           </visual>
