Commit message: Add also DiffBot working

File: ros2_control_demo_description/urdf/diffbot/diffbot.urdf.xacro (robot description, xacro)
@@ -27,5 +27,5 @@
         <box size="${base_width} ${base_length} ${base_height}"/>
       </geometry>
-      <material name="blue"/>
+      <material name="orange"/>
     </visual>
     <inertial>

File: ros2_control_demo_description/urdf/diffbot/diffbot_system.ros2_control.xacro (robot description, xacro)
@@ -1,5 +1,5 @@
 <?xml version="1.0"?>
 <robot xmlns:xacro="http://www.ros.org/wiki/xacro">
-  <xacro:macro name="rrbot_system_position_only" params="name prefix use_fake_hardware:=^|true fake_sensor_commands:=^|false slowdown:=2.0">
+  <xacro:macro name="diffbot_system" params="name prefix use_fake_hardware:=^|false fake_sensor_commands:=^|false slowdown:=2.0">
     <ros2_control name="${name}" type="system">
       <hardware>

File: ros2_control_demo_description/urdf/diffbot_system.urdf.xacro (robot description, xacro)
@@ -2,8 +2,13 @@
 <!-- Basic differential drive mobile base -->
 <!--
-Copied and modified from ROS1 example:
+Copied and modified from ROS1 example -
 https://github.com/ros-simulation/gazebo_ros_demos/blob/kinetic-devel/diffbot_description/urdf/diffbot.xacro
 -->
-<robot xmlns:xacro="http://www.ros.org/wiki/xacro" name="2dof_robot">
+<robot xmlns:xacro="http://www.ros.org/wiki/xacro" name="diffdrive_robot">
+  <xacro:arg name="use_sim" default="false" />
+  <!-- Enable setting arguments from the launch file -->
+  <xacro:arg name="use_fake_hardware" default="true" />
+  <xacro:arg name="fake_sensor_commands" default="false" />
+  <xacro:arg name="prefix" default="" />
   <xacro:include filename="$(find ros2_control_demo_description)/urdf/diffbot/diffbot.urdf.xacro" />
   <!-- Import all Gazebo-customization elements, including Gazebo colors -->
@@ -13,6 +18,9 @@
   <!-- Import diffbot ros2_control description -->
   <xacro:include filename="$(find ros2_control_demo_description)/urdf/diffbot/diffbot_system.ros2_control.xacro" />
-  <xacro:diffbot prefix="" />
-  <xacro:diffbot_gazebo prefix="" />
-  <xacro:diffbot_system name="DiffBotSystem" prefix="" />
+  <xacro:diffbot prefix="$(arg prefix)" />
+  <xacro:diffbot_gazebo prefix="$(arg prefix)" />
+  <xacro:diffbot_system
+    name="DiffBotSystem" prefix="$(arg prefix)"
+    use_fake_hardware="$(arg use_fake_hardware)"
+    fake_sensor_commands="$(arg fake_sensor_commands)"/>
 </robot>
