Commit message: Test and correct diffbot robot view launch.

File: ros2_control_demo_description/diffbot_description/urdf/diffbot_description.urdf.xacro (robot description, xacro)
@@ -23,5 +23,5 @@
     </collision>
     <visual>
-      <origin xyz="0 0 0" rpy="0 0 0"/>
+      <origin xyz="0 0 ${base_height/2}" rpy="0 0 0"/>
       <geometry>
         <box size="${base_width} ${base_length} ${base_height}"/>
