Commit message: Replace use_sim with use_gazebo

File: ros2_control_demo_description/diffbot_description/urdf/diffbot_system.urdf.xacro (robot description, xacro)
@@ -6,5 +6,5 @@
 -->
 <robot xmlns:xacro="http://www.ros.org/wiki/xacro" name="diffdrive_robot">
-  <xacro:arg name="use_sim" default="false" />
+  <xacro:arg name="use_gazebo" default="false" />
   <!-- Enable setting arguments from the launch file -->
   <xacro:arg name="use_fake_hardware" default="true" />

File: ros2_control_demo_description/rrbot_description/ros2_control/external_rrbot_force_torque_sensor.ros2_control.xacro (robot description, xacro)
@@ -1,5 +1,5 @@
 <?xml version="1.0"?>
 <robot xmlns:xacro="http://www.ros.org/wiki/xacro">
-  <xacro:macro name="external_rrbot_force_torque_sensor" params="name prefix use_sim:=^|false use_fake_hardware:=^|true fake_sensor_commands:=^|false">
+  <xacro:macro name="external_rrbot_force_torque_sensor" params="name prefix use_gazebo:=^|false use_fake_hardware:=^|true fake_sensor_commands:=^|false">
     <ros2_control name="${name}" type="sensor">
       <hardware>

File: ros2_control_demo_description/rrbot_description/ros2_control/rrbot_modular_actuators.ros2_control.xacro (robot description, xacro)
@@ -1,5 +1,5 @@
 <?xml version="1.0"?>
 <robot xmlns:xacro="http://www.ros.org/wiki/xacro">
-  <xacro:macro name="rrbot_modular_actuators" params="name prefix use_sim:=^|false slowdown:=2.0">
+  <xacro:macro name="rrbot_modular_actuators" params="name prefix use_gazebo:=^|false slowdown:=2.0">
     <ros2_control name="RRBotModularJoint1" type="actuator">
       <hardware>

File: ros2_control_demo_description/rrbot_description/ros2_control/rrbot_system_multi_interface.ros2_control.xacro (robot description, xacro)
@@ -1,12 +1,12 @@
 <?xml version="1.0"?>
 <robot xmlns:xacro="http://www.ros.org/wiki/xacro">
-  <xacro:macro name="rrbot_system_multi_interface" params="name prefix use_sim:=^|false use_fake_hardware:=^|true fake_sensor_commands:=^|false slowdown:=2.0">
+  <xacro:macro name="rrbot_system_multi_interface" params="name prefix use_gazebo:=^|false use_fake_hardware:=^|true fake_sensor_commands:=^|false slowdown:=2.0">
     <ros2_control name="${name}" type="system">
-      <xacro:if value="$(arg use_sim)">
+      <xacro:if value="$(arg use_gazebo)">
         <hardware>
           <plugin>gazebo_ros2_control/GazeboSystem</plugin>
         </hardware>
       </xacro:if>
-      <xacro:unless value="$(arg use_sim)">
+      <xacro:unless value="$(arg use_gazebo)">
         <hardware>
           <xacro:if value="${use_fake_hardware}">

File: ros2_control_demo_description/rrbot_description/ros2_control/rrbot_system_position_only.ros2_control.xacro (robot description, xacro)
@@ -1,12 +1,12 @@
 <?xml version="1.0"?>
 <robot xmlns:xacro="http://www.ros.org/wiki/xacro">
-  <xacro:macro name="rrbot_system_position_only" params="name prefix use_sim:=^|false use_fake_hardware:=^|true fake_sensor_commands:=^|false slowdown:=2.0">
+  <xacro:macro name="rrbot_system_position_only" params="name prefix use_gazebo:=^|false use_fake_hardware:=^|true fake_sensor_commands:=^|false slowdown:=2.0">
     <ros2_control name="${name}" type="system">
-      <xacro:if value="$(arg use_sim)">
+      <xacro:if value="$(arg use_gazebo)">
         <hardware>
           <plugin>gazebo_ros2_control/GazeboSystem</plugin>
         </hardware>
       </xacro:if>
-      <xacro:unless value="$(arg use_sim)">
+      <xacro:unless value="$(arg use_gazebo)">
         <hardware>
           <xacro:if value="${use_fake_hardware}">

File: ros2_control_demo_description/rrbot_description/ros2_control/rrbot_system_with_sensor.ros2_control.xacro (robot description, xacro)
@@ -1,5 +1,5 @@
 <?xml version="1.0"?>
 <robot xmlns:xacro="http://www.ros.org/wiki/xacro">
-  <xacro:macro name="rrbot_system_with_sensor" params="name prefix use_sim:=^|false use_fake_hardware:=^|true fake_sensor_commands:=^|false slowdown:=2.0">
+  <xacro:macro name="rrbot_system_with_sensor" params="name prefix use_gazebo:=^|false use_fake_hardware:=^|true fake_sensor_commands:=^|false slowdown:=2.0">
     <ros2_control name="${name}" type="system">
       <hardware>

File: ros2_control_demo_description/rrbot_description/urdf/rrbot_modular_actuators.urdf.xacro (robot description, xacro)
@@ -6,5 +6,5 @@
 -->
 <robot xmlns:xacro="http://www.ros.org/wiki/xacro" name="2dof_robot">
-  <xacro:arg name="use_sim" default="false" />
+  <xacro:arg name="use_gazebo" default="false" />
   <!-- Enable setting arguments from the launch file -->
   <xacro:arg name="prefix" default="" />

File: ros2_control_demo_description/rrbot_description/urdf/rrbot_system_multi_interface.urdf.xacro (robot description, xacro)
@@ -6,5 +6,5 @@
 -->
 <robot xmlns:xacro="http://www.ros.org/wiki/xacro" name="2dof_robot">
-  <xacro:arg name="use_sim" default="false" />
+  <xacro:arg name="use_gazebo" default="false" />
   <!-- Enable setting arguments from the launch file -->
   <xacro:arg name="use_fake_hardware" default="false" />

File: ros2_control_demo_description/rrbot_description/urdf/rrbot_system_position_only.urdf.xacro (robot description, xacro)
@@ -6,5 +6,5 @@
 -->
 <robot xmlns:xacro="http://www.ros.org/wiki/xacro" name="2dof_robot">
-  <xacro:arg name="use_sim" default="false" />
+  <xacro:arg name="use_gazebo" default="false" />
   <!-- Enable setting arguments from the launch file -->
   <xacro:arg name="use_fake_hardware" default="false" />

File: ros2_control_demo_description/rrbot_description/urdf/rrbot_system_with_external_sensor.urdf.xacro (robot description, xacro)
@@ -6,5 +6,5 @@
 -->
 <robot xmlns:xacro="http://www.ros.org/wiki/xacro" name="2dof_robot">
-  <xacro:arg name="use_sim" default="false" />
+  <xacro:arg name="use_gazebo" default="false" />
   <!-- Enable setting arguments from the launch file -->
   <xacro:arg name="use_fake_hardware" default="true" />

File: ros2_control_demo_description/rrbot_description/urdf/rrbot_system_with_sensor.urdf.xacro (robot description, xacro)
@@ -6,5 +6,5 @@
 -->
 <robot xmlns:xacro="http://www.ros.org/wiki/xacro" name="2dof_robot">
-  <xacro:arg name="use_sim" default="false" />
+  <xacro:arg name="use_gazebo" default="false" />
   <!-- Enable setting arguments from the launch file -->
   <xacro:arg name="use_fake_hardware" default="false" />
