Commit message: rrbot launch file
Signed-off-by: Karsten Knese <Karsten1987@users.noreply.github.com>

File: ros2_control_demo_description/rrbot_description/urdf/rrbot.urdf.xacro (robot description, xacro)
@@ -5,5 +5,5 @@
   <xacro:property name="mass" value="1" /> <!-- arbitrary value for mass -->
   <xacro:property name="width" value="0.1" /> <!-- Square dimensions (widthxwidth) of beams -->
-  <xacro:property name="height1" value="0.2" /> <!-- Link 1 -->
+  <xacro:property name="height1" value="2" /> <!-- Link 1 -->
   <xacro:property name="height2" value="1" /> <!-- Link 2 -->
   <xacro:property name="height3" value="1" /> <!-- Link 3 -->
@@ -126,5 +126,5 @@
             <origin xyz="0 0 0" rpy="0 0 0"/>
             <geometry>
-              <mesh filename="package://ros2_control_demo_description/meshes/hokuyo.dae"/>
+              <mesh filename="package://rrbot_description/meshes/hokuyo.dae"/>
             </geometry>
           </visual>

File: ros2_control_demo_description/rrbot_description/urdf/rrbot_system_position_only.urdf.xacro (robot description, xacro)
@@ -8,16 +8,16 @@
   <xacro:arg name="use_sim" default="false" />
   <!-- Enable setting arguments from the launch file -->
-  <xacro:arg name="use_fake_hardware" default="true" />
+  <xacro:arg name="use_fake_hardware" default="false" />
   <xacro:arg name="fake_sensor_commands" default="false" />
   <xacro:arg name="prefix" default="" />
   <xacro:arg name="slowdown" default="2.0" />
   <!-- Import RRBot macro -->
-  <xacro:include filename="$(find ros2_control_demo_description)/urdf/rrbot/rrbot.urdf.xacro" />
+  <xacro:include filename="$(find rrbot_description)/urdf/rrbot.urdf.xacro" />
   <!-- Import all Gazebo-customization elements, including Gazebo colors -->
-  <xacro:include filename="$(find ros2_control_demo_description)/urdf/rrbot/gazebo/rrbot.gazebo.xacro" />
+  <xacro:include filename="$(find rrbot_description)/gazebo/rrbot.gazebo.xacro" />
   <!-- Import Rviz colors -->
-  <xacro:include filename="$(find ros2_control_demo_description)/urdf/rrbot/gazebo/rrbot.materials.xacro" />
+  <xacro:include filename="$(find rrbot_description)/gazebo/rrbot.materials.xacro" />
   <!-- Import RRBot ros2_control description -->
-  <xacro:include filename="$(find ros2_control_demo_description)/urdf/rrbot/ros2_control/rrbot_system_position_only.ros2_control.xacro" />
+  <xacro:include filename="$(find rrbot_description)/ros2_control/rrbot_system_position_only.ros2_control.xacro" />
   <!-- Used for fixing robot -->
   <link name="world"/>

Commit message: Add RRBot minimal example.

File: ros2_control_demo_description/rrbot_description/urdf/rrbot.urdf.xacro (robot description, xacro)
@@ -1,176 +1,25 @@
 <?xml version="1.0"?>
-<robot xmlns:xacro="http://www.ros.org/wiki/xacro">
-  <xacro:macro name="rrbot" params="parent prefix *origin">
-  <!-- Constants for robot dimensions -->
-  <xacro:property name="mass" value="1" /> <!-- arbitrary value for mass -->
-  <xacro:property name="width" value="0.1" /> <!-- Square dimensions (widthxwidth) of beams -->
-  <xacro:property name="height1" value="2" /> <!-- Link 1 -->
-  <xacro:property name="height2" value="1" /> <!-- Link 2 -->
-  <xacro:property name="height3" value="1" /> <!-- Link 3 -->
-  <xacro:property name="camera_link" value="0.05" /> <!-- Size of square 'camera' box -->
-  <xacro:property name="axel_offset" value="0.05" /> <!-- Space btw top of beam and the each joint -->
-  <joint name="${prefix}base_joint" type="fixed">
-    <xacro:insert_block name="origin" />
-    <parent link="${parent}"/>
-    <child link="${prefix}base_link" />
-  </joint>
-  <!-- Base Link -->
-  <link name="${prefix}base_link">
-    <collision>
-      <origin xyz="0 0 ${height1/2}" rpy="0 0 0"/>
-      <geometry>
-        <box size="${width} ${width} ${height1}"/>
-      </geometry>
-    </collision>
-    <visual>
-      <origin xyz="0 0 ${height1/2}" rpy="0 0 0"/>
-      <geometry>
-        <box size="${width} ${width} ${height1}"/>
-      </geometry>
-      <material name="orange"/>
-    </visual>
-    <inertial>
-      <origin xyz="0 0 ${height1/2}" rpy="0 0 0"/>
-      <mass value="${mass}"/>
-      <inertia
-        ixx="${mass / 12.0 * (width*width + height1*height1)}" ixy="0.0" ixz="0.0"
-        iyy="${mass / 12.0 * (height1*height1 + width*width)}" iyz="0.0"
-        izz="${mass / 12.0 * (width*width + width*width)}"/>
-      </inertial>
-    </link>
-    <joint name="${prefix}joint1" type="continuous">
-      <parent link="${prefix}base_link"/>
-      <child link="${prefix}link1"/>
-      <origin xyz="0 ${width} ${height1 - axel_offset}" rpy="0 0 0"/>
-      <axis xyz="0 1 0"/>
-      <dynamics damping="0.7"/>
-    </joint>
-    <!-- Middle Link -->
-    <link name="${prefix}link1">
-      <collision>
-        <origin xyz="0 0 ${height2/2 - axel_offset}" rpy="0 0 0"/>
-        <geometry>
-          <box size="${width} ${width} ${height2}"/>
-        </geometry>
-      </collision>
-      <visual>
-        <origin xyz="0 0 ${height2/2 - axel_offset}" rpy="0 0 0"/>
-        <geometry>
-          <box size="${width} ${width} ${height2}"/>
-        </geometry>
-        <material name="yellow"/>
-      </visual>
-      <inertial>
-        <origin xyz="0 0 ${height2/2 - axel_offset}" rpy="0 0 0"/>
-        <mass value="${mass}"/>
-        <inertia
-          ixx="${mass / 12.0 * (width*width + height2*height2)}" ixy="0.0" ixz="0.0"
-          iyy="${mass / 12.0 * (height2*height2 + width*width)}" iyz="0.0"
-          izz="${mass / 12.0 * (width*width + width*width)}"/>
-        </inertial>
-      </link>
-      <joint name="${prefix}joint2" type="continuous">
-        <parent link="${prefix}link1"/>
-        <child link="${prefix}link2"/>
-        <origin xyz="0 ${width} ${height2 - axel_offset*2}" rpy="0 0 0"/>
-        <axis xyz="0 1 0"/>
-        <dynamics damping="0.7"/>
-      </joint>
-      <!-- Top Link -->
-      <link name="${prefix}link2">
-        <collision>
-          <origin xyz="0 0 ${height3/2 - axel_offset}" rpy="0 0 0"/>
-          <geometry>
-            <box size="${width} ${width} ${height3}"/>
-          </geometry>
-        </collision>
-        <visual>
-          <origin xyz="0 0 ${height3/2 - axel_offset}" rpy="0 0 0"/>
-          <geometry>
-            <box size="${width} ${width} ${height3}"/>
-          </geometry>
-          <material name="orange"/>
-        </visual>
-        <inertial>
-          <origin xyz="0 0 ${height3/2 - axel_offset}" rpy="0 0 0"/>
-          <mass value="${mass}"/>
-          <inertia
-            ixx="${mass / 12.0 * (width*width + height3*height3)}" ixy="0.0" ixz="0.0"
-            iyy="${mass / 12.0 * (height3*height3 + width*width)}" iyz="0.0"
-            izz="${mass / 12.0 * (width*width + width*width)}"/>
-          </inertial>
-        </link>
-        <joint name="${prefix}tool_joint" type="fixed">
-          <origin xyz="0 0 1" rpy="0 0 0" />
-          <parent link="${prefix}link2"/>
-          <child link="${prefix}tool_link" />
-        </joint>
-        <!-- Tool Link -->
-        <link name="${prefix}tool_link">
-        </link>
-        <joint name="${prefix}hokuyo_joint" type="fixed">
-          <axis xyz="0 1 0" />
-          <origin xyz="0 0 ${height3 - axel_offset/2}" rpy="0 0 0"/>
-          <parent link="${prefix}link2"/>
-          <child link="${prefix}hokuyo_link"/>
-        </joint>
-        <!-- Hokuyo Laser -->
-        <link name="${prefix}hokuyo_link">
-          <collision>
-            <origin xyz="0 0 0" rpy="0 0 0"/>
-            <geometry>
-              <box size="0.1 0.1 0.1"/>
-            </geometry>
-          </collision>
-          <visual>
-            <origin xyz="0 0 0" rpy="0 0 0"/>
-            <geometry>
-              <mesh filename="package://rrbot_description/meshes/hokuyo.dae"/>
-            </geometry>
-          </visual>
-          <inertial>
-            <mass value="1e-5" />
-            <origin xyz="0 0 0" rpy="0 0 0"/>
-            <inertia ixx="1e-6" ixy="0" ixz="0" iyy="1e-6" iyz="0" izz="1e-6" />
-          </inertial>
-        </link>
-        <joint name="${prefix}camera_joint" type="fixed">
-          <axis xyz="0 1 0" />
-          <origin xyz="${camera_link} 0 ${height3 - axel_offset*2}" rpy="0 0 0"/>
-          <parent link="${prefix}link2"/>
-          <child link="${prefix}camera_link"/>
-        </joint>
-        <!-- Camera -->
-        <link name="${prefix}camera_link">
-          <collision>
-            <origin xyz="0 0 0" rpy="0 0 0"/>
-            <geometry>
-              <box size="${camera_link} ${camera_link} ${camera_link}"/>
-            </geometry>
-          </collision>
-          <visual>
-            <origin xyz="0 0 0" rpy="0 0 0"/>
-            <geometry>
-              <box size="${camera_link} ${camera_link} ${camera_link}"/>
-            </geometry>
-            <material name="red"/>
-          </visual>
-          <inertial>
-            <mass value="1e-5" />
-            <origin xyz="0 0 0" rpy="0 0 0"/>
-            <inertia ixx="1e-6" ixy="0" ixz="0" iyy="1e-6" iyz="0" izz="1e-6" />
-          </inertial>
-        </link>
-        <!-- generate an optical frame http://www.ros.org/reps/rep-0103.html#suffix-frames
-        so that ros and opencv can operate on the camera frame correctly -->
-        <joint name="${prefix}camera_optical_joint" type="fixed">
-          <!-- these values have to be these values otherwise the gazebo camera image
-          won't be aligned properly with the frame it is supposedly originating from -->
-          <origin xyz="0 0 0" rpy="${-pi/2} 0 ${-pi/2}"/>
-          <parent link="${prefix}camera_link"/>
-          <child link="${prefix}camera_link_optical"/>
-        </joint>
-        <link name="${prefix}camera_link_optical">
-        </link>
-  </xacro:macro>
+<!-- Revolute-Revolute Manipulator -->
+<!--
+Copied and modified from ROS1 example -
+https://github.com/ros-simulation/gazebo_ros_demos/blob/kinetic-devel/rrbot_description/urdf/rrbot.xacro
+-->
+<robot xmlns:xacro="http://www.ros.org/wiki/xacro" name="2dof_robot">
+  <xacro:arg name="prefix" default="" />
+  <!-- Import RRBot macro -->
+  <xacro:include filename="$(find rrbot_description)/urdf/rrbot_description.urdf.xacro" />
+  <!-- Import Rviz colors -->
+  <xacro:include filename="$(find rrbot_description)/gazebo/rrbot.materials.xacro" />
+  <!-- Import RRBot ros2_control description -->
+  <xacro:include filename="$(find rrbot_description)/ros2_control/rrbot.ros2_control.xacro" />
+  <!-- Used for fixing robot -->
+  <link name="world"/>
+  <gazebo reference="world">
+    <static>true</static>
+  </gazebo>
+  <xacro:rrbot parent="world" prefix="$(arg prefix)">
+    <origin xyz="0 0 0" rpy="0 0 0" />
+  </xacro:rrbot>
+  <xacro:rrbot_ros2_control
+    name="RRBot" prefix="$(arg prefix)" />
 </robot>

File: ros2_control_demo_description/rrbot_description/urdf/rrbot_system_multi_interface.urdf.xacro (robot description, xacro)
@@ -8,16 +8,16 @@
   <xacro:arg name="use_sim" default="false" />
   <!-- Enable setting arguments from the launch file -->
-  <xacro:arg name="use_fake_hardware" default="true" />
+  <xacro:arg name="use_fake_hardware" default="false" />
   <xacro:arg name="fake_sensor_commands" default="false" />
   <xacro:arg name="prefix" default="" />
   <xacro:arg name="slowdown" default="2.0" />
   <!-- Import RRBot macro -->
-  <xacro:include filename="$(find rrbot_description)/urdf/rrbot/rrbot.urdf.xacro" />
+  <xacro:include filename="$(find rrbot_description)/urdf/rrbot_description.urdf.xacro" />
   <!-- Import all Gazebo-customization elements, including Gazebo colors -->
-  <xacro:include filename="$(find rrbot_description)/urdf/rrbot/gazebo/rrbot.gazebo.xacro" />
+  <xacro:include filename="$(find rrbot_description)/gazebo/rrbot.gazebo.xacro" />
   <!-- Import Rviz colors -->
-  <xacro:include filename="$(find rrbot_description)/urdf/rrbot/gazebo/rrbot.materials.xacro" />
+  <xacro:include filename="$(find rrbot_description)/gazebo/rrbot.materials.xacro" />
   <!-- Import RRBot ros2_control description -->
-  <xacro:include filename="$(find rrbot_description)/urdf/rrbot/ros2_control/rrbot_system_multi_interface.ros2_control.xacro" />
+  <xacro:include filename="$(find rrbot_description)/ros2_control/rrbot_system_multi_interface.ros2_control.xacro" />
   <!-- Used for fixing robot -->
   <link name="world"/>
