Commit message: Finalize example with prefix and multi controller manager.

File: ros2_control_demo_description/rrbot_description/urdf/rrbot_system_position_only.urdf.xacro (robot description, xacro)
@@ -26,5 +26,5 @@
   </gazebo>
   <xacro:rrbot parent="world" prefix="$(arg prefix)">
-    <origin xyz="0 0 0" rpy="0 0 0" />
+    <origin xyz="1 1 0" rpy="0 0 0" />
   </xacro:rrbot>
   <xacro:rrbot_gazebo prefix="$(arg prefix)" />
