Commit message: Bugfix: Do not ignore prefix argument for joint names.

File: ros2_control_demo_description/rrbot_description/ros2_control/external_rrbot_force_torque_sensor.ros2_control.xacro (robot description, xacro)
@@ -16,5 +16,5 @@
         </xacro:unless>
       </hardware>
-      <sensor name="tcp_fts_sensor">
+      <sensor name="${prefix}tcp_fts_sensor">
         <state_interface name="force.x"/>
         <state_interface name="force.y"/>

File: ros2_control_demo_description/rrbot_description/ros2_control/rrbot_system_position_only.ros2_control.xacro (robot description, xacro)
@@ -23,5 +23,5 @@
         </hardware>
       </xacro:unless>
-      <joint name="joint1">
+      <joint name="${prefix}joint1">
         <command_interface name="position">
           <param name="min">-1</param>
@@ -30,5 +30,5 @@
         <state_interface name="position"/>
       </joint>
-      <joint name="joint2">
+      <joint name="${prefix}joint2">
         <command_interface name="position">
           <param name="min">-1</param>

File: ros2_control_demo_description/rrbot_description/ros2_control/rrbot_system_with_sensor.ros2_control.xacro (robot description, xacro)
@@ -17,5 +17,5 @@
         </xacro:unless>
       </hardware>
-      <joint name="joint1">
+      <joint name="${prefix}joint1">
         <command_interface name="position">
           <param name="min">-1</param>
@@ -24,5 +24,5 @@
         <state_interface name="position"/>
       </joint>
-      <joint name="joint2">
+      <joint name="${prefix}joint2">
         <command_interface name="position">
           <param name="min">-1</param>
@@ -31,5 +31,5 @@
         <state_interface name="position"/>
       </joint>
-      <sensor name="tcp_fts_sensor">
+      <sensor name="${prefix}tcp_fts_sensor">
         <state_interface name="force.x"/>
         <state_interface name="torque.z"/>
