Commit message: Add disable_commands to parameter propagation pipeline.

File: ros2_control_demo_description/rrbot_description/ros2_control/rrbot_system_position_only.ros2_control.xacro (robot description, xacro)
@@ -1,5 +1,5 @@
 <?xml version="1.0"?>
 <robot xmlns:xacro="http://www.ros.org/wiki/xacro">
-  <xacro:macro name="rrbot_system_position_only" params="name prefix use_sim:=^|false use_fake_hardware:=^|true fake_sensor_commands:=^|false slowdown:=2.0">
+  <xacro:macro name="rrbot_system_position_only" params="name prefix use_sim:=^|false use_fake_hardware:=^|true fake_sensor_commands:=^|false slowdown:=2.0 disable_commands:=^|false">
     <ros2_control name="${name}" type="system">
       <xacro:if value="$(arg use_sim)">
@@ -14,4 +14,5 @@
             <param name="fake_sensor_commands">${fake_sensor_commands}</param>
             <param name="state_following_offset">0.0</param>
+            <param name="disable_commands">${disable_commands}</param>
           </xacro:if>
           <xacro:unless value="${use_fake_hardware}">

Commit message: Bugfix: Do not ignore prefix argument for joint names.

File: ros2_control_demo_description/rrbot_description/ros2_control/rrbot_system_position_only.ros2_control.xacro (robot description, xacro)
@@ -23,5 +23,5 @@
         </hardware>
       </xacro:unless>
-      <joint name="joint1">
+      <joint name="${prefix}joint1">
         <command_interface name="position">
           <param name="min">-1</param>
@@ -30,5 +30,5 @@
         <state_interface name="position"/>
       </joint>
-      <joint name="joint2">
+      <joint name="${prefix}joint2">
         <command_interface name="position">
           <param name="min">-1</param>
