Commit message: Add disable command param. Add action client test for jtc.

File: ros2_control_demo_description/rrbot_description/ros2_control/rrbot_system_multi_interface.ros2_control.xacro (robot description, xacro)
@@ -1,5 +1,5 @@
 <?xml version="1.0"?>
 <robot xmlns:xacro="http://www.ros.org/wiki/xacro">
-  <xacro:macro name="rrbot_system_multi_interface" params="name prefix use_sim:=^|false use_fake_hardware:=^|true fake_sensor_commands:=^|false slowdown:=2.0">
+  <xacro:macro name="rrbot_system_multi_interface" params="name prefix use_sim:=^|false use_fake_hardware:=^|true fake_sensor_commands:=^|false slowdown:=2.0 disable_commands:=^|false">
     <ros2_control name="${name}" type="system">
       <xacro:if value="$(arg use_sim)">
@@ -14,4 +14,5 @@
             <param name="fake_sensor_commands">${fake_sensor_commands}</param>
             <param name="state_following_offset">0.0</param>
+            <param name="disable_commands">${disable_commands}</param>
           </xacro:if>
           <xacro:unless value="${use_fake_hardware}">

File: ros2_control_demo_description/rrbot_description/urdf/rrbot_system_multi_interface.urdf.xacro (robot description, xacro)
@@ -33,4 +33,5 @@
     use_fake_hardware="$(arg use_fake_hardware)"
     fake_sensor_commands="$(arg fake_sensor_commands)"
-    slowdown="$(arg slowdown)" />
+    slowdown="$(arg slowdown)"
+    disable_commands="$(arg disable_commands)" />
 </robot>
