Commit message: Corrected and finilized example 5

File: ros2_control_demo_description/rrbot_description/ros2_control/rrbot_modular_actuators.ros2_control.xacro (robot description, xacro)
@@ -1,5 +1,5 @@
 <?xml version="1.0"?>
 <robot xmlns:xacro="http://www.ros.org/wiki/xacro">
-  <xacro:macro name="rrbot_system_separate_actuators" params="name prefix use_sim:=^|false use_fake_hardware:=^|true fake_sensor_commands:=^|false slowdown:=2.0">
+  <xacro:macro name="rrbot_modular_actuators" params="name prefix use_sim:=^|false slowdown:=2.0">
     <ros2_control name="RRBotModularJoint1" type="actuator">
       <hardware>
@@ -11,6 +11,6 @@
       <joint name="joint1">
         <command_interface name="position">
-          <param name="min">-1</param>
-          <param name="max">1</param>
+          <param name="min">-100</param>
+          <param name="max">100</param>
         </command_interface>
         <state_interface name="position"/>
@@ -26,6 +26,6 @@
       <joint name="joint2">
         <command_interface name="position">
-          <param name="min">-1</param>
-          <param name="max">1</param>
+          <param name="min">-100</param>
+          <param name="max">100</param>
         </command_interface>
         <state_interface name="position"/>

File: ros2_control_demo_description/rrbot_description/urdf/rrbot_modular_actuators.urdf.xacro (robot description, xacro)
@@ -8,5 +8,4 @@
   <xacro:arg name="use_sim" default="false" />
   <!-- Enable setting arguments from the launch file -->
-  <xacro:arg name="use_fake_hardware" default="false" />
   <xacro:arg name="prefix" default="" />
   <xacro:arg name="slowdown" default="2.0" />
@@ -18,5 +17,5 @@
   <xacro:include filename="$(find rrbot_description)/gazebo/rrbot.materials.xacro" />
   <!-- Import RRBot ros2_control description -->
-  <xacro:include filename="$(find rrbot_description)/ros2_control/rrbot_system_separate_actuators.ros2_control.xacro" />
+  <xacro:include filename="$(find rrbot_description)/ros2_control/rrbot_modular_actuators.ros2_control.xacro" />
   <!-- Used for fixing robot -->
   <link name="world"/>
@@ -28,7 +27,6 @@
   </xacro:rrbot>
   <xacro:rrbot_gazebo prefix="$(arg prefix)" />
-  <xacro:rrbot_system_separate_actuators
+  <xacro:rrbot_modular_actuators
     name="RRBotModularJoint" prefix="$(arg prefix)"
-    use_fake_hardware="$(arg use_fake_hardware)"
     slowdown="$(arg slowdown)" />
 </robot>

Commit message: Fix rest two files.

File: ros2_control_demo_description/rrbot_description/ros2_control/rrbot_modular_actuators.ros2_control.xacro (robot description, xacro)
@@ -9,5 +9,5 @@
         <param name="example_param_hw_slowdown">${slowdown}</param>
       </hardware>
-      <joint name="joint1">
+      <joint name="${prefix}joint1">
         <command_interface name="position">
           <param name="min">-100</param>
@@ -24,5 +24,5 @@
         <param name="example_param_hw_slowdown">${slowdown}</param>
       </hardware>
-      <joint name="joint2">
+      <joint name="${prefix}joint2">
         <command_interface name="position">
           <param name="min">-100</param>

File: ros2_control_demo_description/rrbot_description/ros2_control/rrbot_system_multi_interface.ros2_control.xacro (robot description, xacro)
@@ -23,5 +23,5 @@
         </hardware>
       </xacro:unless>
-      <joint name="joint1">
+      <joint name="${prefix}joint1">
         <command_interface name="position">
           <param name="min">-1</param>
@@ -40,5 +40,5 @@
         <state_interface name="acceleration"/>
       </joint>
-      <joint name="joint2">
+      <joint name="${prefix}joint2">
         <command_interface name="position">
           <param name="min">-1</param>
