Commit message: rename transmissions ros2_control macro

File: ros2_control_demo_description/rrbot_description/ros2_control/rrbot_transmissions_system_position_only.ros2_control.xacro (robot description, xacro)
@@ -1,5 +1,5 @@
 <?xml version="1.0"?>
 <robot xmlns:xacro="http://www.ros.org/wiki/xacro">
-  <xacro:macro name="rrbot_system_position_only" params="name prefix use_gazebo:=^|false use_fake_hardware:=^|true mock_sensor_commands:=^|false slowdown:=2.0">
+  <xacro:macro name="rrbot_transmissions_system_position_only" params="name prefix use_gazebo:=^|false use_fake_hardware:=^|true mock_sensor_commands:=^|false slowdown:=2.0">
     <ros2_control name="${name}" type="system">
       <xacro:if value="$(arg use_gazebo)">

File: ros2_control_demo_description/rrbot_description/urdf/rrbot_transmissions_system_position_only.urdf.xacro (robot description, xacro)
@@ -29,5 +29,5 @@
   </xacro:rrbot>
   <xacro:rrbot_gazebo prefix="$(arg prefix)" />
-  <xacro:rrbot_system_position_only
+  <xacro:rrbot_transmissions_system_position_only
     name="RRBotTransmissionsSystemPositionOnly" prefix="$(arg prefix)"
     use_fake_hardware="$(arg use_fake_hardware)"
