Commit message: added visual meshes for robot

File: 6_dof_robot/urdf/inc/create_link.xacro (robot description, xacro)
@@ -11,5 +11,5 @@
                 <origin xyz="${xyz_offset}" rpy="${rpy_offset}"/>
                 <geometry>
-                    <mesh filename="package://${mesh_package}/meshes/visual/${mesh_name}.stl"/>
+                    <mesh filename="package://${mesh_package}/meshes/visual/${mesh_name}.dae"/>
                 </geometry>
             </visual>
