Commit message: added trajectory generation

File: robot_6_dof/urdf/robot_6_dof.urdf (robot description, URDF)
Before this commit: robot robot_6_dof, 10 links, 9 joints
Joints:
- joint joint-tool: origin xyz=0 0 0 rpy=0 0 0 -> xyz=0 0 .185 rpy=0 0 0

File: robot_6_dof/urdf/robot_6_dof.urdf.xacro (robot description, xacro)
@@ -114,5 +114,5 @@
     <parent link="ft_frame"/>
     <child link="tool0"/>
-    <origin xyz="0 0 0" rpy="0 0 0"/>
+    <origin xyz="0 0 .185" rpy="0 0 0"/>
   </joint>
   <!-- ros2 control tag -->
