Commit message: working restructured repo

File: robot_6_dof/robot_description/urdf/robot_6_dof.urdf (robot description, URDF)
Before this commit: robot robot_6_dof, 10 links, 9 joints
Links:
- link base_link: geometry collision mesh filename=package://robot_description/meshes/collision/link_0.stl; visual mesh filename=package://robot_description/meshes/visual/link_0.dae
- link link_1: geometry collision mesh filename=package://robot_description/meshes/collision/link_1.stl; visual mesh filename=package://robot_description/meshes/visual/link_1.dae
- link link_2: geometry collision mesh filename=package://robot_description/meshes/collision/link_2.stl; visual mesh filename=package://robot_description/meshes/visual/link_2.dae
- link link_3: geometry collision mesh filename=package://robot_description/meshes/collision/link_3.stl; visual mesh filename=package://robot_description/meshes/visual/link_3.dae
- link link_4: geometry collision mesh filename=package://robot_description/meshes/collision/link_4.stl; visual mesh filename=package://robot_description/meshes/visual/link_4.dae
- link link_5: geometry collision mesh filename=package://robot_description/meshes/collision/link_5.stl; visual mesh filename=package://robot_description/meshes/visual/link_5.dae
- link link_6: geometry collision mesh filename=package://robot_description/meshes/collision/link_6.stl; visual mesh filename=package://robot_description/meshes/visual/link_6.dae

File: robot_6_dof/robot_description/urdf/robot_6_dof.urdf.xacro (robot description, xacro)
@@ -2,5 +2,5 @@
 <robot xmlns:xacro="http://wiki.ros.org/xacro" name="robot_6_dof">
   <!-- helper macro -->
-  <xacro:include filename="$(find robot_6_dof)/urdf/inc/create_link.xacro"/>
+  <xacro:include filename="$(find robot_description)/urdf/inc/create_link.xacro"/>
   <!-- create link fixed to the "world" -->
   <link name="world"/>
@@ -9,5 +9,5 @@
       xyz_offset="0 0 0"
       rpy_offset="0 0 0"
-      mesh_package="robot_6_dof"
+      mesh_package="robot_description"
       mesh_name="link_0"
   />
@@ -16,5 +16,5 @@
       xyz_offset="0 0 0"
       rpy_offset="0 0 0"
-      mesh_package="robot_6_dof"
+      mesh_package="robot_description"
       mesh_name="link_1"
   />
@@ -23,5 +23,5 @@
       xyz_offset="0 0 0"
       rpy_offset="0 0 0"
-      mesh_package="robot_6_dof"
+      mesh_package="robot_description"
       mesh_name="link_2"
   />
@@ -30,5 +30,5 @@
       xyz_offset="0 0 0"
       rpy_offset="0 0 0"
-      mesh_package="robot_6_dof"
+      mesh_package="robot_description"
       mesh_name="link_3"
   />
@@ -37,5 +37,5 @@
       xyz_offset="0 0 0"
       rpy_offset="0 0 0"
-      mesh_package="robot_6_dof"
+      mesh_package="robot_description"
       mesh_name="link_4"
   />
@@ -44,5 +44,5 @@
       xyz_offset="0 0 0"
       rpy_offset="0 0 0"
-      mesh_package="robot_6_dof"
+      mesh_package="robot_description"
       mesh_name="link_5"
   />
@@ -51,5 +51,5 @@
       xyz_offset="0 0 0"
       rpy_offset="0 0 0"
-      mesh_package="robot_6_dof"
+      mesh_package="robot_description"
       mesh_name="link_6"
   />
