Commit message: clang-format

File: r6bot/r6bot_description/urdf/inc/create_link.xacro (robot description, xacro)
@@ -1,5 +1,5 @@
 <?xml version="1.0"?>
 <robot xmlns:xacro="http://wiki.ros.org/xacro">
-    <xacro:macro name="create_link" params="
+  <xacro:macro name="create_link" params="
         link_name
         xyz_offset
@@ -7,22 +7,22 @@
         mesh_package
         mesh_name">
-        <link name="${link_name}">
-            <visual>
-                <origin xyz="${xyz_offset}" rpy="${rpy_offset}"/>
-                <geometry>
-                    <mesh filename="package://${mesh_package}/meshes/visual/${mesh_name}.dae"/>
-                </geometry>
-            </visual>
-            <collision>
-                <origin xyz="${xyz_offset}" rpy="${rpy_offset}"/>
-                <geometry>
-                    <mesh filename="package://${mesh_package}/meshes/collision/${mesh_name}.stl"/>
-                </geometry>
-            </collision>
-            <inertial>
-                <mass value="1"/>
-                <inertia ixx="1.0" ixy="0.0" ixz="0.0" iyy="1.0" iyz="0.0" izz="1.0"/>
-            </inertial>
-        </link>
-    </xacro:macro>
+    <link name="${link_name}">
+      <visual>
+        <origin xyz="${xyz_offset}" rpy="${rpy_offset}"/>
+        <geometry>
+          <mesh filename="package://${mesh_package}/meshes/visual/${mesh_name}.dae"/>
+        </geometry>
+      </visual>
+      <collision>
+        <origin xyz="${xyz_offset}" rpy="${rpy_offset}"/>
+        <geometry>
+          <mesh filename="package://${mesh_package}/meshes/collision/${mesh_name}.stl"/>
+        </geometry>
+      </collision>
+      <inertial>
+        <mass value="1"/>
+        <inertia ixx="1.0" ixy="0.0" ixz="0.0" iyy="1.0" iyz="0.0" izz="1.0"/>
+      </inertial>
+    </link>
+  </xacro:macro>
 </robot>

File: r6bot/r6bot_description/urdf/r6bot.urdf.xacro (robot description, xacro)
@@ -69,5 +69,5 @@
     <origin xyz="0 0 0.061584" rpy="0 0 0"/>
     <axis xyz="0 0 1"/>
-    <limit effort="1000.0" lower="${-pi}" upper="${pi}" velocity="2.5" />
+    <limit effort="1000.0" lower="${-pi}" upper="${pi}" velocity="2.5"/>
   </joint>
   <joint name="joint_2" type="revolute">
@@ -76,5 +76,5 @@
     <origin xyz="-0.101717 0 0.182284" rpy="${-pi/2} -${pi/3} ${pi/2}"/>
     <axis xyz="0 0 1"/>
-    <limit effort="1000.0" lower="${-pi}" upper="${pi}" velocity="2.5" />
+    <limit effort="1000.0" lower="${-pi}" upper="${pi}" velocity="2.5"/>
   </joint>
   <joint name="joint_3" type="revolute">
@@ -83,5 +83,5 @@
     <origin xyz="0.685682 0 0.041861" rpy="0 ${pi} ${pi+pi/2}"/>
     <axis xyz="0 0 1"/>
-    <limit effort="1000.0" lower="${-pi}" upper="${pi}" velocity="2.5" />
+    <limit effort="1000.0" lower="${-pi}" upper="${pi}" velocity="2.5"/>
   </joint>
   <joint name="joint_4" type="revolute">
@@ -90,5 +90,5 @@
     <origin xyz="0.518777 0 0.067458" rpy="0 ${pi} ${pi+pi/6}"/>
     <axis xyz="0 0 1"/>
-    <limit effort="1000.0" lower="${-pi}" upper="${pi}" velocity="2.5" />
+    <limit effort="1000.0" lower="${-pi}" upper="${pi}" velocity="2.5"/>
   </joint>
   <joint name="joint_5" type="revolute">
@@ -97,5 +97,5 @@
     <origin xyz="0.112654 0 0.110903" rpy="${pi/2} ${pi} ${pi/2}"/>
     <axis xyz="0 0 1"/>
-    <limit effort="1000.0" lower="${-pi}" upper="${pi}" velocity="2.5" />
+    <limit effort="1000.0" lower="${-pi}" upper="${pi}" velocity="2.5"/>
   </joint>
   <joint name="joint_6" type="revolute">
@@ -104,5 +104,5 @@
     <origin xyz="-0.085976 0 0.133436" rpy="0 ${-pi/2} 0"/>
     <axis xyz="0 0 1"/>
-    <limit effort="1000.0" lower="${-pi}" upper="${pi}" velocity="2.5" />
+    <limit effort="1000.0" lower="${-pi}" upper="${pi}" velocity="2.5"/>
   </joint>
   <joint name="joint-ft_frame" type="fixed">
