Commit message: Fixed the example and improved docs

File: example_5/description/urdf/rrbot_system_with_external_sensor.urdf.xacro (robot description, xacro)
@@ -22,5 +22,5 @@
   <link name="world"/>
   <xacro:rrbot parent="world" prefix="$(arg prefix)">
-    <origin xyz="0 0 0" rpy="0 0 0" />
+    <origin xyz="1 1 0" rpy="0 0 0" />
   </xacro:rrbot>
   <xacro:rrbot_system_position_only
