Commit message: Fix rviz

File: example_6/description/urdf/rrbot_description.urdf.xacro (robot description, xacro)
@@ -126,5 +126,5 @@
             <origin xyz="0 0 0" rpy="0 0 0"/>
             <geometry>
-              <mesh filename="package://rrbot_description/meshes/hokuyo.dae"/>
+              <mesh filename="package://ros2_control_demo_example_6/meshes/hokuyo.dae"/>
             </geometry>
           </visual>
