Commit message: Initial commit for example_8

File: example_8/description/ros2_control/rrbot_transmissions_system_position_only.ros2_control.xacro (robot description, xacro)
@@ -1,8 +1,8 @@
 <?xml version="1.0"?>
 <robot xmlns:xacro="http://www.ros.org/wiki/xacro">
-  <xacro:macro name="rrbot_transmissions_system_position_only" params="name prefix use_gazebo:=^|false use_fake_hardware:=^|true mock_sensor_commands:=^|false slowdown:=2.0">
+  <xacro:macro name="rrbot_transmissions_system_position_only" params="name prefix slowdown:=2.0">
     <ros2_control name="${name}" type="system">
       <hardware>
-        <plugin>ros2_control_demo_hardware/RRBotTransmissionsSystemPositionOnlyHardware</plugin>
+        <plugin>ros2_control_demo_example_8/RRBotTransmissionsSystemPositionOnlyHardware</plugin>
         <param name="actuator_slowdown">${slowdown}</param>
       </hardware>

File: example_8/description/urdf/rrbot_transmissions_system_position_only.urdf.xacro (robot description, xacro)
@@ -10,9 +10,9 @@
   <xacro:arg name="slowdown" default="100.0" />
   <!-- Import RRBot macro -->
-  <xacro:include filename="$(find rrbot_description)/urdf/rrbot_description.urdf.xacro" />
+  <xacro:include filename="$(find ros2_control_demo_example_8)/urdf/rrbot_description.urdf.xacro" />
   <!-- Import Rviz colors -->
-  <xacro:include filename="$(find rrbot_description)/gazebo/rrbot.materials.xacro" />
+  <xacro:include filename="$(find ros2_control_demo_example_8)/urdf/rrbot.materials.xacro" />
   <!-- Import RRBot ros2_control description -->
-  <xacro:include filename="$(find rrbot_description)/ros2_control/rrbot_transmissions_system_position_only.ros2_control.xacro" />
+  <xacro:include filename="$(find ros2_control_demo_example_8)/ros2_control/rrbot_transmissions_system_position_only.ros2_control.xacro" />
   <!-- Used for fixing robot -->
   <link name="world"/>
@@ -25,6 +25,4 @@
   <xacro:rrbot_transmissions_system_position_only
     name="RRBotTransmissionsSystemPositionOnly" prefix="$(arg prefix)"
-    use_fake_hardware="$(arg use_fake_hardware)"
-    mock_sensor_commands="$(arg mock_sensor_commands)"
     slowdown="$(arg slowdown)" />
 </robot>
