Commit message: Remove gazebo xacro/launch-file parameters

File: example_1/description/urdf/rrbot.urdf.xacro (robot description, xacro)
@@ -15,7 +15,4 @@
   <!-- Used for fixing robot -->
   <link name="world"/>
-  <gazebo reference="world">
-    <static>true</static>
-  </gazebo>
   <xacro:rrbot parent="world" prefix="$(arg prefix)">
     <origin xyz="0 0 0" rpy="0 0 0" />

File: example_3/description/ros2_control/rrbot_system_multi_interface.ros2_control.xacro (robot description, xacro)
@@ -1,26 +1,19 @@
 <?xml version="1.0"?>
 <robot xmlns:xacro="http://www.ros.org/wiki/xacro">
-  <xacro:macro name="rrbot_system_multi_interface" params="name prefix use_gazebo:=^|false use_fake_hardware:=^|true mock_sensor_commands:=^|false slowdown:=2.0">
+  <xacro:macro name="rrbot_system_multi_interface" params="name prefix use_fake_hardware:=^|true mock_sensor_commands:=^|false slowdown:=2.0">
     <ros2_control name="${name}" type="system">
-      <xacro:if value="$(arg use_gazebo)">
-        <hardware>
-          <plugin>gazebo_ros2_control/GazeboSystem</plugin>
-        </hardware>
-      </xacro:if>
-      <xacro:unless value="$(arg use_gazebo)">
-        <hardware>
-          <xacro:if value="${use_fake_hardware}">
-            <plugin>mock_components/GenericSystem</plugin>
-            <param name="mock_sensor_commands">${mock_sensor_commands}</param>
-            <param name="state_following_offset">0.0</param>
-          </xacro:if>
-          <xacro:unless value="${use_fake_hardware}">
-            <plugin>ros2_control_demo_example_3/RRBotSystemMultiInterfaceHardware</plugin>
-            <param name="example_param_hw_start_duration_sec">0.0</param>
-            <param name="example_param_hw_stop_duration_sec">3.0</param>
-            <param name="example_param_hw_slowdown">${slowdown}</param>
-          </xacro:unless>
-        </hardware>
-      </xacro:unless>
+      <hardware>
+        <xacro:if value="${use_fake_hardware}">
+          <plugin>mock_components/GenericSystem</plugin>
+          <param name="mock_sensor_commands">${mock_sensor_commands}</param>
+          <param name="state_following_offset">0.0</param>
+        </xacro:if>
+        <xacro:unless value="${use_fake_hardware}">
+          <plugin>ros2_control_demo_example_3/RRBotSystemMultiInterfaceHardware</plugin>
+          <param name="example_param_hw_start_duration_sec">0.0</param>
+          <param name="example_param_hw_stop_duration_sec">3.0</param>
+          <param name="example_param_hw_slowdown">${slowdown}</param>
+        </xacro:unless>
+      </hardware>
       <joint name="${prefix}joint1">
         <command_interface name="position">

File: example_3/description/urdf/rrbot_system_multi_interface.urdf.xacro (robot description, xacro)
@@ -6,5 +6,4 @@
 -->
 <robot xmlns:xacro="http://www.ros.org/wiki/xacro" name="2dof_robot">
-  <xacro:arg name="use_gazebo" default="false" />
   <!-- Enable setting arguments from the launch file -->
   <xacro:arg name="use_fake_hardware" default="false" />
@@ -20,7 +19,4 @@
   <!-- Used for fixing robot -->
   <link name="world"/>
-  <gazebo reference="world">
-    <static>true</static>
-  </gazebo>
   <xacro:rrbot parent="world" prefix="$(arg prefix)">
     <origin xyz="0 0 0" rpy="0 0 0" />

File: example_4/description/ros2_control/rrbot_system_with_sensor.ros2_control.xacro (robot description, xacro)
@@ -1,5 +1,5 @@
 <?xml version="1.0"?>
 <robot xmlns:xacro="http://www.ros.org/wiki/xacro">
-  <xacro:macro name="rrbot_system_with_sensor" params="name prefix use_gazebo:=^|false use_fake_hardware:=^|true mock_sensor_commands:=^|false slowdown:=2.0">
+  <xacro:macro name="rrbot_system_with_sensor" params="name prefix use_fake_hardware:=^|true mock_sensor_commands:=^|false slowdown:=2.0">
     <ros2_control name="${name}" type="system">
       <hardware>

File: example_4/description/urdf/rrbot_system_with_sensor.urdf.xacro (robot description, xacro)
@@ -6,5 +6,4 @@
 -->
 <robot xmlns:xacro="http://www.ros.org/wiki/xacro" name="2dof_robot">
-  <xacro:arg name="use_gazebo" default="false" />
   <!-- Enable setting arguments from the launch file -->
   <xacro:arg name="use_fake_hardware" default="false" />
@@ -20,7 +19,4 @@
   <!-- Used for fixing robot -->
   <link name="world"/>
-  <gazebo reference="world">
-    <static>true</static>
-  </gazebo>
   <xacro:rrbot parent="world" prefix="$(arg prefix)">
     <origin xyz="0 0 0" rpy="0 0 0" />

File: example_5/description/ros2_control/external_rrbot_force_torque_sensor.ros2_control.xacro (robot description, xacro)
@@ -1,5 +1,5 @@
 <?xml version="1.0"?>
 <robot xmlns:xacro="http://www.ros.org/wiki/xacro">
-  <xacro:macro name="external_rrbot_force_torque_sensor" params="name prefix use_gazebo:=^|false use_fake_hardware:=^|true mock_sensor_commands:=^|false">
+  <xacro:macro name="external_rrbot_force_torque_sensor" params="name prefix use_fake_hardware:=^|true mock_sensor_commands:=^|false">
     <ros2_control name="${name}" type="sensor">
       <hardware>

File: example_5/description/ros2_control/rrbot_system_position_only.ros2_control.xacro (robot description, xacro)
@@ -1,26 +1,19 @@
 <?xml version="1.0"?>
 <robot xmlns:xacro="http://www.ros.org/wiki/xacro">
-  <xacro:macro name="rrbot_system_position_only" params="name prefix use_gazebo:=^|false use_fake_hardware:=^|true mock_sensor_commands:=^|false slowdown:=2.0">
+  <xacro:macro name="rrbot_system_position_only" params="name prefix use_fake_hardware:=^|true mock_sensor_commands:=^|false slowdown:=2.0">
     <ros2_control name="${name}" type="system">
-      <xacro:if value="$(arg use_gazebo)">
-        <hardware>
-          <plugin>gazebo_ros2_control/GazeboSystem</plugin>
-        </hardware>
-      </xacro:if>
-      <xacro:unless value="$(arg use_gazebo)">
-        <hardware>
-          <xacro:if value="${use_fake_hardware}">
-            <plugin>mock_components/GenericSystem</plugin>
-            <param name="mock_sensor_commands">${mock_sensor_commands}</param>
-            <param name="state_following_offset">0.0</param>
-          </xacro:if>
-          <xacro:unless value="${use_fake_hardware}">
-            <plugin>ros2_control_demo_example_5/RRBotSystemPositionOnlyHardware</plugin>
-            <param name="example_param_hw_start_duration_sec">0.0</param>
-            <param name="example_param_hw_stop_duration_sec">3.0</param>
-            <param name="example_param_hw_slowdown">${slowdown}</param>
-          </xacro:unless>
-        </hardware>
-      </xacro:unless>
+      <hardware>
+        <xacro:if value="${use_fake_hardware}">
+          <plugin>mock_components/GenericSystem</plugin>
+          <param name="mock_sensor_commands">${mock_sensor_commands}</param>
+          <param name="state_following_offset">0.0</param>
+        </xacro:if>
+        <xacro:unless value="${use_fake_hardware}">
+          <plugin>ros2_control_demo_example_5/RRBotSystemPositionOnlyHardware</plugin>
+          <param name="example_param_hw_start_duration_sec">0.0</param>
+          <param name="example_param_hw_stop_duration_sec">3.0</param>
+          <param name="example_param_hw_slowdown">${slowdown}</param>
+        </xacro:unless>
+      </hardware>
       <joint name="${prefix}joint1">
         <command_interface name="position">

File: example_5/description/urdf/rrbot_system_with_external_sensor.urdf.xacro (robot description, xacro)
@@ -6,5 +6,4 @@
 -->
 <robot xmlns:xacro="http://www.ros.org/wiki/xacro" name="2dof_robot">
-  <xacro:arg name="use_gazebo" default="false" />
   <!-- Enable setting arguments from the launch file -->
   <xacro:arg name="use_fake_hardware" default="true" />
@@ -22,7 +21,4 @@
   <!-- Used for fixing robot -->
   <link name="world"/>
-  <gazebo reference="world">
-    <static>true</static>
-  </gazebo>
   <xacro:rrbot parent="world" prefix="$(arg prefix)">
     <origin xyz="0 0 0" rpy="0 0 0" />

File: example_6/description/ros2_control/rrbot_modular_actuators.ros2_control.xacro (robot description, xacro)
@@ -1,5 +1,5 @@
 <?xml version="1.0"?>
 <robot xmlns:xacro="http://www.ros.org/wiki/xacro">
-  <xacro:macro name="rrbot_modular_actuators" params="name prefix use_gazebo:=^|false slowdown:=2.0">
+  <xacro:macro name="rrbot_modular_actuators" params="name prefix slowdown:=2.0">
     <ros2_control name="RRBotModularJoint1" type="actuator">
       <hardware>

File: example_6/description/urdf/rrbot_modular_actuators.urdf.xacro (robot description, xacro)
@@ -6,5 +6,4 @@
 -->
 <robot xmlns:xacro="http://www.ros.org/wiki/xacro" name="2dof_robot">
-  <xacro:arg name="use_gazebo" default="false" />
   <!-- Enable setting arguments from the launch file -->
   <xacro:arg name="prefix" default="" />
@@ -18,7 +17,4 @@
   <!-- Used for fixing robot -->
   <link name="world"/>
-  <gazebo reference="world">
-    <static>true</static>
-  </gazebo>
   <xacro:rrbot parent="world" prefix="$(arg prefix)">
     <origin xyz="0 0 0" rpy="0 0 0" />

File: example_8/description/urdf/rrbot_transmissions_system_position_only.urdf.xacro (robot description, xacro)
@@ -17,7 +17,4 @@
   <!-- Used for fixing robot -->
   <link name="world"/>
-  <gazebo reference="world">
-    <static>true</static>
-  </gazebo>
   <xacro:rrbot parent="world" prefix="$(arg prefix)">
     <origin xyz="0 0 0" rpy="0 0 0" />
