Commit message: Rename "fake_hardware" to "mock_hardware".

File: example_3/description/ros2_control/rrbot_system_multi_interface.ros2_control.xacro (robot description, xacro)
@@ -1,13 +1,13 @@
 <?xml version="1.0"?>
 <robot xmlns:xacro="http://www.ros.org/wiki/xacro">
-  <xacro:macro name="rrbot_system_multi_interface" params="name prefix use_fake_hardware:=^|true mock_sensor_commands:=^|false slowdown:=2.0">
+  <xacro:macro name="rrbot_system_multi_interface" params="name prefix use_mock_hardware:=^|true mock_sensor_commands:=^|false slowdown:=2.0">
     <ros2_control name="${name}" type="system">
       <hardware>
-        <xacro:if value="${use_fake_hardware}">
+        <xacro:if value="${use_mock_hardware}">
           <plugin>mock_components/GenericSystem</plugin>
           <param name="mock_sensor_commands">${mock_sensor_commands}</param>
           <param name="state_following_offset">0.0</param>
         </xacro:if>
-        <xacro:unless value="${use_fake_hardware}">
+        <xacro:unless value="${use_mock_hardware}">
           <plugin>ros2_control_demo_example_3/RRBotSystemMultiInterfaceHardware</plugin>
           <param name="example_param_hw_start_duration_sec">0.0</param>

File: example_3/description/urdf/rrbot_system_multi_interface.urdf.xacro (robot description, xacro)
@@ -7,5 +7,5 @@
 <robot xmlns:xacro="http://www.ros.org/wiki/xacro" name="2dof_robot">
   <!-- Enable setting arguments from the launch file -->
-  <xacro:arg name="use_fake_hardware" default="false" />
+  <xacro:arg name="use_mock_hardware" default="false" />
   <xacro:arg name="mock_sensor_commands" default="false" />
   <xacro:arg name="prefix" default="" />
@@ -24,5 +24,5 @@
   <xacro:rrbot_system_multi_interface
     name="RRBotSystemMultiInterface" prefix="$(arg prefix)"
-    use_fake_hardware="$(arg use_fake_hardware)"
+    use_mock_hardware="$(arg use_mock_hardware)"
     mock_sensor_commands="$(arg mock_sensor_commands)"
     slowdown="$(arg slowdown)" />

File: example_4/description/ros2_control/rrbot_system_with_sensor.ros2_control.xacro (robot description, xacro)
@@ -1,13 +1,13 @@
 <?xml version="1.0"?>
 <robot xmlns:xacro="http://www.ros.org/wiki/xacro">
-  <xacro:macro name="rrbot_system_with_sensor" params="name prefix use_fake_hardware:=^|true mock_sensor_commands:=^|false slowdown:=2.0">
+  <xacro:macro name="rrbot_system_with_sensor" params="name prefix use_mock_hardware:=^|true mock_sensor_commands:=^|false slowdown:=2.0">
     <ros2_control name="${name}" type="system">
       <hardware>
-        <xacro:if value="${use_fake_hardware}">
+        <xacro:if value="${use_mock_hardware}">
           <plugin>mock_components/GenericSystem</plugin>
           <param name="mock_sensor_commands">${mock_sensor_commands}</param>
           <param name="state_following_offset">0.0</param>
         </xacro:if>
-        <xacro:unless value="${use_fake_hardware}">
+        <xacro:unless value="${use_mock_hardware}">
           <plugin>ros2_control_demo_example_4/RRBotSystemWithSensorHardware</plugin>
           <param name="example_param_hw_start_duration_sec">0.0</param>

File: example_4/description/urdf/rrbot_system_with_sensor.urdf.xacro (robot description, xacro)
@@ -7,5 +7,5 @@
 <robot xmlns:xacro="http://www.ros.org/wiki/xacro" name="2dof_robot">
   <!-- Enable setting arguments from the launch file -->
-  <xacro:arg name="use_fake_hardware" default="false" />
+  <xacro:arg name="use_mock_hardware" default="false" />
   <xacro:arg name="mock_sensor_commands" default="false" />
   <xacro:arg name="prefix" default="" />
@@ -24,5 +24,5 @@
   <xacro:rrbot_system_with_sensor
     name="RRBotSystemWithSensor" prefix="$(arg prefix)"
-    use_fake_hardware="$(arg use_fake_hardware)"
+    use_mock_hardware="$(arg use_mock_hardware)"
     mock_sensor_commands="$(arg mock_sensor_commands)"
     slowdown="$(arg slowdown)" />

File: example_5/description/ros2_control/external_rrbot_force_torque_sensor.ros2_control.xacro (robot description, xacro)
@@ -1,13 +1,13 @@
 <?xml version="1.0"?>
 <robot xmlns:xacro="http://www.ros.org/wiki/xacro">
-  <xacro:macro name="external_rrbot_force_torque_sensor" params="name prefix use_fake_hardware:=^|true mock_sensor_commands:=^|false">
+  <xacro:macro name="external_rrbot_force_torque_sensor" params="name prefix use_mock_hardware:=^|true mock_sensor_commands:=^|false">
     <ros2_control name="${name}" type="sensor">
       <hardware>
-        <xacro:if value="${use_fake_hardware}">
+        <xacro:if value="${use_mock_hardware}">
           <plugin>mock_components/GenericSystem</plugin>
           <param name="mock_sensor_commands">${mock_sensor_commands}</param>
           <param name="state_following_offset">0.0</param>
         </xacro:if>
-        <xacro:unless value="${use_fake_hardware}">
+        <xacro:unless value="${use_mock_hardware}">
           <plugin>ros2_control_demo_example_5/ExternalRRBotForceTorqueSensorHardware</plugin>
           <param name="example_param_hw_start_duration_sec">0.0</param>

File: example_5/description/ros2_control/rrbot_system_position_only.ros2_control.xacro (robot description, xacro)
@@ -1,13 +1,13 @@
 <?xml version="1.0"?>
 <robot xmlns:xacro="http://www.ros.org/wiki/xacro">
-  <xacro:macro name="rrbot_system_position_only" params="name prefix use_fake_hardware:=^|true mock_sensor_commands:=^|false slowdown:=2.0">
+  <xacro:macro name="rrbot_system_position_only" params="name prefix use_mock_hardware:=^|true mock_sensor_commands:=^|false slowdown:=2.0">
     <ros2_control name="${name}" type="system">
       <hardware>
-        <xacro:if value="${use_fake_hardware}">
+        <xacro:if value="${use_mock_hardware}">
           <plugin>mock_components/GenericSystem</plugin>
           <param name="mock_sensor_commands">${mock_sensor_commands}</param>
           <param name="state_following_offset">0.0</param>
         </xacro:if>
-        <xacro:unless value="${use_fake_hardware}">
+        <xacro:unless value="${use_mock_hardware}">
           <plugin>ros2_control_demo_example_5/RRBotSystemPositionOnlyHardware</plugin>
           <param name="example_param_hw_start_duration_sec">0.0</param>

File: example_5/description/urdf/rrbot_system_with_external_sensor.urdf.xacro (robot description, xacro)
@@ -7,5 +7,5 @@
 <robot xmlns:xacro="http://www.ros.org/wiki/xacro" name="2dof_robot">
   <!-- Enable setting arguments from the launch file -->
-  <xacro:arg name="use_fake_hardware" default="true" />
+  <xacro:arg name="use_mock_hardware" default="true" />
   <xacro:arg name="mock_sensor_commands" default="false" />
   <xacro:arg name="prefix" default="" />
@@ -26,10 +26,10 @@
   <xacro:rrbot_system_position_only
     name="RRBotSystemPositionOnly" prefix="$(arg prefix)"
-    use_fake_hardware="$(arg use_fake_hardware)"
+    use_mock_hardware="$(arg use_mock_hardware)"
     mock_sensor_commands="$(arg mock_sensor_commands)"
     slowdown="$(arg slowdown)" />
   <xacro:external_rrbot_force_torque_sensor
     name="ExternalRRBotFTSensor" prefix="$(arg prefix)"
-    use_fake_hardware="$(arg use_fake_hardware)"
+    use_mock_hardware="$(arg use_mock_hardware)"
     mock_sensor_commands="$(arg mock_sensor_commands)" />
 </robot>
