Commit message: Fix rviz

File: example_4/description/urdf/rrbot_description.urdf.xacro (robot description, xacro)
@@ -126,5 +126,5 @@
             <origin xyz="0 0 0" rpy="0 0 0"/>
             <geometry>
-              <mesh filename="package://rrbot_description/meshes/hokuyo.dae"/>
+              <mesh filename="package://ros2_control_demo_example_4/meshes/hokuyo.dae"/>
             </geometry>
           </visual>

Commit message: Readd missing joints for tool_link

File: example_4/description/urdf/rrbot_description.urdf.xacro (robot description, xacro)
@@ -100,4 +100,12 @@
           </inertial>
         </link>
+  <joint name="${prefix}tool_joint" type="fixed">
+    <origin xyz="0 0 1" rpy="0 0 0" />
+    <parent link="${prefix}link2"/>
+    <child link="${prefix}tool_link" />
+  </joint>
+  <!-- Tool Link -->
+  <link name="${prefix}tool_link">
+  </link>
   </xacro:macro>
 </robot>

File: example_5/description/urdf/rrbot_description.urdf.xacro (robot description, xacro)
@@ -100,4 +100,12 @@
           </inertial>
         </link>
+        <joint name="${prefix}tool_joint" type="fixed">
+          <origin xyz="0 0 1" rpy="0 0 0" />
+          <parent link="${prefix}link2"/>
+          <child link="${prefix}tool_link" />
+        </joint>
+        <!-- Tool Link -->
+        <link name="${prefix}tool_link">
+        </link>
   </xacro:macro>
 </robot>
