Commit message: Remove Gazebo simulator

File: example_9/description/ros2_control/rrbot.ros2_control.xacro (robot description, xacro)
@@ -1,5 +1,5 @@
 <?xml version="1.0"?>
 <robot xmlns:xacro="http://www.ros.org/wiki/xacro">
-  <xacro:macro name="rrbot_ros2_control" params="name prefix use_gazebo_classic:=^|false use_gazebo:=^|false">
+  <xacro:macro name="rrbot_ros2_control" params="name prefix use_gazebo_classic:=^|false">
     <ros2_control name="${name}" type="system">
       <hardware>
@@ -8,13 +8,8 @@
         </xacro:if>
         <xacro:unless value="${use_gazebo_classic}">
-          <xacro:if value="${use_gazebo}">
-            <plugin>gz_ros2_control/GazeboSimSystem</plugin>
-          </xacro:if>
-          <xacro:unless value="${use_gazebo}">
-            <plugin>ros2_control_demo_example_9/RRBotSystemPositionOnlyHardware</plugin>
-            <param name="example_param_hw_start_duration_sec">0</param>
-            <param name="example_param_hw_stop_duration_sec">3.0</param>
-            <param name="example_param_hw_slowdown">100</param>
-          </xacro:unless>
+          <plugin>ros2_control_demo_example_9/RRBotSystemPositionOnlyHardware</plugin>
+          <param name="example_param_hw_start_duration_sec">0</param>
+          <param name="example_param_hw_stop_duration_sec">3.0</param>
+          <param name="example_param_hw_slowdown">100</param>
         </xacro:unless>
       </hardware>

File: example_9/description/urdf/rrbot.urdf.xacro (robot description, xacro)
@@ -8,5 +8,4 @@
   <xacro:arg name="prefix" default="" />
   <xacro:arg name="use_gazebo_classic" default="false" />
-  <xacro:arg name="use_gazebo" default="false" />
   <!-- Import RRBot macro -->
   <xacro:include filename="$(find ros2_control_demo_example_9)/urdf/rrbot_description.urdf.xacro" />
@@ -21,5 +20,5 @@
   </xacro:rrbot>
   <xacro:rrbot_ros2_control
-    name="RRBot" prefix="$(arg prefix)" use_gazebo_classic="$(arg use_gazebo_classic)" use_gazebo="$(arg use_gazebo)"/>
+    name="RRBot" prefix="$(arg prefix)" use_gazebo_classic="$(arg use_gazebo_classic)"/>
   <xacro:if value="$(arg use_gazebo_classic)">
     <!-- Import Gazebo Classic definitions + plugin -->
@@ -27,11 +26,3 @@
     <xacro:rrbot_gazebo prefix="$(arg prefix)"/>
   </xacro:if>
-  <xacro:if value="$(arg use_gazebo)">
-    <gazebo>
-      <!-- load Gazebo plugin -->
-      <plugin filename="libgz_ros2_control-system.so" name="gz_ros2_control::GazeboSimROS2ControlPlugin">
-        <parameters>$(find ros2_control_demo_example_9)/config/rrbot_controllers.yaml</parameters>
-      </plugin>
-    </gazebo>
-  </xacro:if>
 </robot>
