Commit message: added controller specific control descriptions

File: example_11/description/ros2_control/carlikebot_ackermann.ros2_control.xacro (robot description, xacro)
@@ -1,8 +1,8 @@
 <?xml version="1.0"?>
 <robot xmlns:xacro="http://www.ros.org/wiki/xacro">
-  <xacro:macro name="diffbot_ros2_control" params="name prefix">
+  <xacro:macro name="carlikebot_ros2_control" params="name prefix">
     <ros2_control name="${name}" type="system">
       <hardware>
-        <plugin>ros2_control_demo_example_2/DiffBotSystemHardware</plugin>
+        <plugin>ros2_control_demo_example_11/CarlikeBotSystemHardware</plugin>
         <param name="example_param_hw_start_duration_sec">0</param>
         <param name="example_param_hw_stop_duration_sec">3.0</param>

File: example_11/description/urdf/carlikebot.urdf.xacro (robot description, xacro)
@@ -1,13 +1,19 @@
 <?xml version="1.0"?>
-<!-- Basic differential drive mobile base -->
-<robot xmlns:xacro="http://www.ros.org/wiki/xacro" name="diffdrive_robot">
+<!-- 4 Wheel Robot with front steering and rear drive -->
+<robot xmlns:xacro="http://www.ros.org/wiki/xacro" name="carlikebot_robot">
   <xacro:arg name="prefix" default="" />
-  <xacro:include filename="$(find ros2_control_demo_example_2)/urdf/diffbot_description.urdf.xacro" />
+  <xacro:arg name="sim" default="false" />
+  <xacro:include filename="$(find ros2_control_demo_example_11)/urdf/carlikebot_description.urdf.xacro" />
   <!-- Import Rviz colors -->
-  <xacro:include filename="$(find ros2_control_demo_example_2)/urdf/diffbot.materials.xacro" />
-  <!-- Import diffbot ros2_control description -->
-  <xacro:include filename="$(find ros2_control_demo_example_2)/ros2_control/diffbot.ros2_control.xacro" />
-  <xacro:diffbot prefix="$(arg prefix)" />
-  <xacro:diffbot_ros2_control
-    name="DiffBot" prefix="$(arg prefix)" />
+  <xacro:include filename="$(find ros2_control_demo_example_11)/urdf/carlikebot.materials.xacro" />
+  <!-- Import carlikebot ros2_control description based on sim arg -->
+  <xacro:if value="$(arg sim)">
+    <xacro:include filename="$(find ros2_control_demo_example_11)/ros2_control/carlikebot_ackermann.ros2_control.xacro" />
+  </xacro:if>
+  <xacro:unless value="$(arg sim)">
+    <xacro:include filename="$(find ros2_control_demo_example_11)/ros2_control/carlikebot_bicycle.ros2_control.xacro" />
+  </xacro:unless>
+  <xacro:carlikebot prefix="$(arg prefix)" />
+  <xacro:carlikebot_ros2_control
+    name="CarlikeBot" prefix="$(arg prefix)" />
 </robot>

File: example_11/description/urdf/carlikebot_description.urdf.xacro (robot description, xacro)
@@ -1,5 +1,5 @@
 <?xml version="1.0"?>
 <robot xmlns:xacro="http://www.ros.org/wiki/xacro">
-  <xacro:macro name="diffbot" params="prefix">
+  <xacro:macro name="carlikebot" params="prefix">
   <!-- Constants for robot dimensions -->
   <xacro:property name="PI" value="3.1415926535897931"/>

Commit message: almost

File: example_11/description/ros2_control/carlikebot_ackermann.ros2_control.xacro (robot description, xacro)
@@ -7,13 +7,20 @@
         <param name="example_param_hw_start_duration_sec">0</param>
         <param name="example_param_hw_stop_duration_sec">3.0</param>
+        <param name="is_simulation">1</param>
       </hardware>
-      <joint name="${prefix}left_wheel_joint">
+      <joint name="${prefix}left_steering_hinge_joint">
+        <command_interface name="position"/>
+        <state_interface name="position"/>
+      </joint>
+      <joint name="${prefix}right_steering_hinge_joint">
+        <command_interface name="position"/>
+        <state_interface name="position"/>
+      </joint>
+      <joint name="${prefix}rear_left_wheel_joint">
         <command_interface name="velocity"/>
-        <state_interface name="position"/>
         <state_interface name="velocity"/>
       </joint>
-      <joint name="${prefix}right_wheel_joint">
+      <joint name="${prefix}rear_right_wheel_joint">
         <command_interface name="velocity"/>
-        <state_interface name="position"/>
         <state_interface name="velocity"/>
       </joint>

File: example_11/description/ros2_control/carlikebot_bicycle.ros2_control.xacro (robot description, xacro)
@@ -5,15 +5,12 @@
       <hardware>
         <plugin>ros2_control_demo_example_11/CarlikeBotSystemHardware</plugin>
-        <param name="example_param_hw_start_duration_sec">0</param>
-        <param name="example_param_hw_stop_duration_sec">3.0</param>
+        <param name="is_simulation">0</param>
       </hardware>
-      <joint name="${prefix}left_wheel_joint">
+      <joint name="${prefix}steering_joint">
+        <command_interface name="position"/>
+        <state_interface name="position"/>
+      </joint>
+      <joint name="${prefix}drive_joint">
         <command_interface name="velocity"/>
-        <state_interface name="position"/>
-        <state_interface name="velocity"/>
-      </joint>
-      <joint name="${prefix}right_wheel_joint">
-        <command_interface name="velocity"/>
-        <state_interface name="position"/>
         <state_interface name="velocity"/>
       </joint>

File: example_11/description/urdf/carlikebot.urdf.xacro (robot description, xacro)
@@ -4,12 +4,13 @@
   <xacro:arg name="prefix" default="" />
   <xacro:arg name="sim" default="false" />
-  <xacro:include filename="$(find ros2_control_demo_example_11)/urdf/carlikebot_description.urdf.xacro" />
   <!-- Import Rviz colors -->
   <xacro:include filename="$(find ros2_control_demo_example_11)/urdf/carlikebot.materials.xacro" />
-  <!-- Import carlikebot ros2_control description based on sim arg -->
+  <!-- Import carlikebot description and ros2_control based on sim arg -->
   <xacro:if value="$(arg sim)">
+    <xacro:include filename="$(find ros2_control_demo_example_11)/urdf/carlikebot_ackermann_description.urdf.xacro" />
     <xacro:include filename="$(find ros2_control_demo_example_11)/ros2_control/carlikebot_ackermann.ros2_control.xacro" />
   </xacro:if>
   <xacro:unless value="$(arg sim)">
+    <xacro:include filename="$(find ros2_control_demo_example_11)/urdf/carlikebot_bicycle_description.urdf.xacro" />
     <xacro:include filename="$(find ros2_control_demo_example_11)/ros2_control/carlikebot_bicycle.ros2_control.xacro" />
   </xacro:unless>

Commit message: inactive ackermann; rear joints missing

File: example_11/description/ros2_control/carlikebot_ackermann.ros2_control.xacro (robot description, xacro)
@@ -9,9 +9,9 @@
         <param name="is_simulation">1</param>
       </hardware>
-      <joint name="${prefix}left_steering_hinge_joint">
+      <joint name="${prefix}left_steering_joint">
         <command_interface name="position"/>
         <state_interface name="position"/>
       </joint>
-      <joint name="${prefix}right_steering_hinge_joint">
+      <joint name="${prefix}right_steering_joint">
         <command_interface name="position"/>
         <state_interface name="position"/>

File: example_11/description/urdf/carlikebot_ackermann_description.urdf.xacro (robot description, xacro)
@@ -75,4 +75,5 @@
       <origin xyz="${base_width/2} -${wheelbase/2} -${base_height/2}" rpy="0 0 0"/>
       <axis xyz="-1 0 0"/>
+      <limit effort="100.0" velocity="100.0"/>
       <dynamics damping="0.2"/>
     </joint>
@@ -102,13 +103,14 @@
     </link>
     <joint name="${prefix}rear_left_wheel_joint" type="continuous">
-      <parent link="${prefix}chassis_link"/>
-      <child link="${prefix}rear_left_wheel"/>
+      <parent link="${prefix}chassis_link" />
+      <child link="${prefix}rear_left_wheel" />
       <origin xyz="-${base_width/2} -${wheelbase/2} -${base_height/2}" rpy="0 0 0"/>
       <axis xyz="-1 0 0"/>
+      <limit effort="100.0" velocity="100.0"/>
       <dynamics damping="0.2"/>
     </joint>
     <!-- front wheels -->
     <!-- front right wheel -->
-    <link name="${prefix}right_steering_hinge">
+    <link name="${prefix}right_steering">
       <collision>
         <origin xyz="0 0 0" rpy="${PI/2} 0 ${PI/2}"/>
@@ -133,13 +135,13 @@
       </inertial>
     </link>
-    <joint name="${prefix}right_steering_hinge_joint" type="revolute">
-      <parent link="${prefix}chassis_link"/>
-      <child link="${prefix}right_steering_hinge"/>
+    <joint name="${prefix}right_steering_joint" type="revolute">
+      <parent link="${prefix}chassis_link" />
+      <child link="${prefix}right_steering" />
       <origin xyz="${base_width/2} ${wheelbase/2} -${base_height/2}" rpy="0 0 0"/>
       <axis xyz="0 0 -1"/>
-      <limit lower="-0.4" upper="0.4" effort="0.0" velocity="0.0"/>
+      <limit lower="-0.4" upper="0.4" effort="100.0" velocity="0.0"/>
       <dynamics damping="0.2"/>
     </joint>
-    <link name="${prefix}left_steering_hinge">
+    <link name="${prefix}left_steering">
       <collision>
         <origin xyz="0 0 0" rpy="${PI/2} 0 ${PI/2}"/>
@@ -164,7 +166,7 @@
       </inertial>
     </link>
-    <joint name="${prefix}left_steering_hinge_joint" type="revolute">
-      <parent link="${prefix}chassis_link"/>
-      <child link="${prefix}left_steering_hinge"/>
+    <joint name="${prefix}left_steering_joint" type="revolute">
+      <parent link="${prefix}chassis_link" />
+      <child link="${prefix}left_steering" />
       <origin xyz="-${base_width/2} ${wheelbase/2} -${base_height/2}" rpy="0 0 0"/>
       <axis xyz="0 0 -1"/>

Commit message: ackermann working

File: example_11/description/ros2_control/carlikebot_ackermann.ros2_control.xacro (robot description, xacro)
@@ -19,8 +19,10 @@
       <joint name="${prefix}rear_left_wheel_joint">
         <command_interface name="velocity"/>
+        <state_interface name="position"/>
         <state_interface name="velocity"/>
       </joint>
       <joint name="${prefix}rear_right_wheel_joint">
         <command_interface name="velocity"/>
+        <state_interface name="position"/>
         <state_interface name="velocity"/>
       </joint>

File: example_11/description/urdf/carlikebot_ackermann_description.urdf.xacro (robot description, xacro)
@@ -19,5 +19,5 @@
       <origin xyz="0 0 0" rpy="0 0 0"/>
       <geometry>
-        <box size="${base_width} ${base_length} ${base_height}"/>
+        <box size="${base_length} ${base_width} ${base_height}"/>
       </geometry>
     </collision>
@@ -25,5 +25,5 @@
       <origin xyz="0 0 0" rpy="0 0 0"/>
       <geometry>
-        <box size="${base_width} ${base_length} ${base_height}"/>
+        <box size="${base_length} ${base_width} ${base_height}"/>
       </geometry>
       <material name="orange"/>
@@ -73,5 +73,5 @@
       <parent link="${prefix}chassis_link"/>
       <child link="${prefix}rear_right_wheel"/>
-      <origin xyz="${base_width/2} -${wheelbase/2} -${base_height/2}" rpy="0 0 0"/>
+      <origin xyz="-${wheelbase/2} ${base_width/2} -${base_height/2}" rpy="0 0 ${PI/2}"/>
       <axis xyz="-1 0 0"/>
       <limit effort="100.0" velocity="100.0"/>
@@ -105,5 +105,5 @@
       <parent link="${prefix}chassis_link" />
       <child link="${prefix}rear_left_wheel" />
-      <origin xyz="-${base_width/2} -${wheelbase/2} -${base_height/2}" rpy="0 0 0"/>
+      <origin xyz="-${wheelbase/2} -${base_width/2} -${base_height/2}" rpy="0 0 ${PI/2}"/>
       <axis xyz="-1 0 0"/>
       <limit effort="100.0" velocity="100.0"/>
@@ -138,6 +138,6 @@
       <parent link="${prefix}chassis_link" />
       <child link="${prefix}right_steering" />
-      <origin xyz="${base_width/2} ${wheelbase/2} -${base_height/2}" rpy="0 0 0"/>
-      <axis xyz="0 0 -1"/>
+      <origin xyz="${wheelbase/2} ${base_width/2} -${base_height/2}" rpy="0 0 ${PI/2}"/>
+      <axis xyz="0 0 1"/>
       <limit lower="-0.4" upper="0.4" effort="100.0" velocity="0.0"/>
       <dynamics damping="0.2"/>
@@ -169,6 +169,6 @@
       <parent link="${prefix}chassis_link" />
       <child link="${prefix}left_steering" />
-      <origin xyz="-${base_width/2} ${wheelbase/2} -${base_height/2}" rpy="0 0 0"/>
-      <axis xyz="0 0 -1"/>
+      <origin xyz="${wheelbase/2} -${base_width/2} -${base_height/2}" rpy="0 0 ${PI/2}"/>
+      <axis xyz="0 0 1"/>
       <limit lower="-0.4" upper="0.4" effort="0.0" velocity="0.0"/>
       <dynamics damping="0.2"/>
