Commit message: added front drive wheels; carlikebot.launch broken

File: example_11/description/ros2_control/carlikebot.ros2_control.xacro (robot description, xacro)
@@ -9,11 +9,19 @@
         <param name="is_simulation">1</param>
       </hardware>
-      <joint name="${prefix}left_steering_joint">
+      <joint name="${prefix}front_left_steering_joint">
         <command_interface name="position"/>
         <state_interface name="position"/>
       </joint>
-      <joint name="${prefix}right_steering_joint">
+      <joint name="${prefix}front_right_steering_joint">
         <command_interface name="position"/>
         <state_interface name="position"/>
+      </joint>
+      <joint name="${prefix}front_left_wheel_joint">
+        <command_interface name="velocity"/>
+        <state_interface name="velocity"/>
+      </joint>
+      <joint name="${prefix}front_right_wheel_joint">
+        <command_interface name="velocity"/>
+        <state_interface name="velocity"/>
       </joint>
       <joint name="${prefix}rear_left_wheel_joint">

File: ros2_control_demo_description/carlikebot/urdf/carlikebot_description.urdf.xacro (robot description, xacro)
@@ -112,6 +112,16 @@
     </joint>
     <!-- front wheels -->
+    <!-- front right steering -->
+    <link name="${prefix}front_right_steering" />
+    <joint name="${prefix}front_right_steering_joint" type="revolute">
+      <parent link="${prefix}chassis_link" />
+      <child link="${prefix}front_right_steering" />
+      <origin xyz="${wheelbase/2} ${base_width/2} -${base_height/2}" rpy="0 0 ${PI/2}"/>
+      <axis xyz="0 0 1"/>
+      <limit lower="-0.4" upper="0.4" effort="100.0" velocity="0.0"/>
+      <dynamics damping="0.2"/>
+    </joint>
     <!-- front right wheel -->
-    <link name="${prefix}right_steering">
+    <link name="${prefix}front_right_wheel">
       <collision>
         <origin xyz="0 0 0" rpy="${PI/2} 0 ${PI/2}"/>
@@ -136,13 +146,24 @@
       </inertial>
     </link>
-    <joint name="${prefix}right_steering_joint" type="revolute">
+    <joint name="${prefix}front_right_wheel_joint" type="continuous">
+      <parent link="${prefix}front_right_steering"/>
+      <child link="${prefix}front_right_wheel"/>
+      <origin xyz="0 0 0" rpy="0 0 0"/>
+      <axis xyz="0 1 0"/>
+      <limit effort="100.0" velocity="100.0"/>
+      <dynamics damping="0.2"/>
+    </joint>
+    <!-- front left steering -->
+    <link name="${prefix}front_left_steering" />
+    <joint name="${prefix}front_left_steering_joint" type="revolute">
       <parent link="${prefix}chassis_link" />
-      <child link="${prefix}right_steering" />
-      <origin xyz="${wheelbase/2} ${base_width/2} -${base_height/2}" rpy="0 0 ${PI/2}"/>
+      <child link="${prefix}front_left_steering" />
+      <origin xyz="${wheelbase/2} -${base_width/2} -${base_height/2}" rpy="0 0 ${PI/2}"/>
       <axis xyz="0 0 1"/>
       <limit lower="-0.4" upper="0.4" effort="100.0" velocity="0.0"/>
       <dynamics damping="0.2"/>
     </joint>
-    <link name="${prefix}left_steering">
+    <!-- front left wheel -->
+    <link name="${prefix}front_left_wheel">
       <collision>
         <origin xyz="0 0 0" rpy="${PI/2} 0 ${PI/2}"/>
@@ -167,10 +188,10 @@
       </inertial>
     </link>
-    <joint name="${prefix}left_steering_joint" type="revolute">
-      <parent link="${prefix}chassis_link" />
-      <child link="${prefix}left_steering" />
-      <origin xyz="${wheelbase/2} -${base_width/2} -${base_height/2}" rpy="0 0 ${PI/2}"/>
-      <axis xyz="0 0 1"/>
-      <limit lower="-0.4" upper="0.4" effort="0.0" velocity="0.0"/>
+    <joint name="${prefix}front_left_wheel_joint" type="continuous">
+      <parent link="${prefix}front_left_steering"/>
+      <child link="${prefix}front_left_wheel"/>
+      <origin xyz="0 0 0" rpy="0 0 0"/>
+      <axis xyz="0 1 0"/>
+      <limit effort="100.0" velocity="100.0"/>
       <dynamics damping="0.2"/>
     </joint>

Commit message: configured base

File: example_11/description/ros2_control/carlikebot.ros2_control.xacro (robot description, xacro)
@@ -9,27 +9,12 @@
         <param name="is_simulation">1</param>
       </hardware>
-      <joint name="${prefix}front_left_steering_joint">
+      <joint name="${prefix}virtual_front_wheel_joint">
         <command_interface name="position"/>
         <state_interface name="position"/>
       </joint>
-      <joint name="${prefix}front_right_steering_joint">
-        <command_interface name="position"/>
-        <state_interface name="position"/>
-      </joint>
-      <joint name="${prefix}front_left_wheel_joint">
+      <joint name="${prefix}virtual_rear_wheel_joint">
         <command_interface name="velocity"/>
         <state_interface name="velocity"/>
-      </joint>
-      <joint name="${prefix}front_right_wheel_joint">
-        <command_interface name="velocity"/>
-        <state_interface name="velocity"/>
-      </joint>
-      <joint name="${prefix}rear_left_wheel_joint">
-        <command_interface name="velocity"/>
-        <state_interface name="velocity"/>
-      </joint>
-      <joint name="${prefix}rear_right_wheel_joint">
-        <command_interface name="velocity"/>
-        <state_interface name="velocity"/>
+        <state_interface name="position"/>
       </joint>
     </ros2_control>

File: ros2_control_demo_description/carlikebot/urdf/carlikebot_description.urdf.xacro (robot description, xacro)
@@ -33,8 +33,8 @@
       <origin xyz="0 0 0" rpy="0 0 0"/>
       <mass value="${base_mass}"/>
-      <inertia
-        ixx="${base_mass / 12.0 * (base_length*base_length + base_height*base_height)}" ixy="0.0" ixz="0.0"
-        iyy="${base_mass / 12.0 * (base_height*base_height + base_width*base_width)}" iyz="0.0"
-        izz="${base_mass / 12.0 * (base_width*base_width + base_length*base_length)}"/>
+        <inertia
+          ixx="0.000270" ixy="0.0" ixz="0.0"
+          iyy="0.000270" iyz="0.0"
+          izz="0.000426"/>
       </inertial>
     </link>
@@ -61,5 +61,5 @@
       <child link="${prefix}virtual_rear_wheel"/>
       <origin xyz="-${wheelbase/2} 0 -${base_height/2}" rpy="0 0 ${PI/2}"/>
-      <axis xyz="-1 0 0"/>
+      <axis xyz="1 0 0"/>
       <limit effort="100.0" velocity="100.0"/>
       <dynamics damping="0.2"/>
@@ -84,7 +84,7 @@
         <mass value="${wheel_mass}"/>
         <inertia
-          ixx="${wheel_mass / 12.0 * (3*wheel_radius + wheel_len*wheel_len)}" ixy="0.0" ixz="0.0"
-          iyy="${wheel_mass / 12.0 * wheel_radius*wheel_radius}" iyz="0.0"
-          izz="${wheel_mass / 12.0 * wheel_radius*wheel_radius}"/>
+          ixx="0.000270" ixy="0.0" ixz="0.0"
+          iyy="0.000270" iyz="0.0"
+          izz="0.000426"/>
       </inertial>
     </link>
@@ -93,5 +93,5 @@
       <child link="${prefix}rear_right_wheel"/>
       <origin xyz="-${wheelbase/2} ${base_width/2} -${base_height/2}" rpy="0 0 ${PI/2}"/>
-      <axis xyz="-1 0 0"/>
+      <axis xyz="1 0 0"/>
       <limit effort="100.0" velocity="100.0"/>
       <dynamics damping="0.2"/>
@@ -117,7 +117,7 @@
           <mass value="${wheel_mass}"/>
           <inertia
-            ixx="${wheel_mass / 12.0 * (3*wheel_radius + wheel_len*wheel_len)}" ixy="0.0" ixz="0.0"
-            iyy="${wheel_mass / 12.0 * wheel_radius*wheel_radius}" iyz="0.0"
-            izz="${wheel_mass / 12.0 * wheel_radius*wheel_radius}"/>
+            ixx="0.000270" ixy="0.0" ixz="0.0"
+            iyy="0.000270" iyz="0.0"
+            izz="0.000426"/>
         </inertial>
     </link>
@@ -126,5 +126,5 @@
       <child link="${prefix}rear_left_wheel" />
       <origin xyz="-${wheelbase/2} -${base_width/2} -${base_height/2}" rpy="0 0 ${PI/2}"/>
-      <axis xyz="-1 0 0"/>
+      <axis xyz="1 0 0"/>
       <limit effort="100.0" velocity="100.0"/>
       <dynamics damping="0.2"/>
@@ -132,5 +132,5 @@
     </joint>
     <!-- front wheels -->
-    <!-- virtual front steering -->
+    <!-- virtual front wheel -->
     <link name="${prefix}virtual_front_wheel">
       <visual>
@@ -150,5 +150,5 @@
       <dynamics damping="0.2"/>
     </joint>
-    <!-- front right steering -->
+    <!-- front right wheel -->
     <link name="${prefix}front_right_wheel">
       <collision>
@@ -169,7 +169,7 @@
         <mass value="${wheel_mass}"/>
         <inertia
-          ixx="${wheel_mass / 12.0 * (3*wheel_radius + wheel_len*wheel_len)}" ixy="0.0" ixz="0.0"
-          iyy="${wheel_mass / 12.0 * wheel_radius*wheel_radius}" iyz="0.0"
-          izz="${wheel_mass / 12.0 * wheel_radius*wheel_radius}"/>
+          ixx="0.000270" ixy="0.0" ixz="0.0"
+          iyy="0.000270" iyz="0.0"
+          izz="0.000426"/>
       </inertial>
     </link>
@@ -202,7 +202,7 @@
         <mass value="${wheel_mass}"/>
         <inertia
-          ixx="${wheel_mass / 12.0 * (3 * wheel_radius + wheel_len * wheel_len)}" ixy="0.0" ixz="0.0"
-          iyy="${wheel_mass / 12.0 * wheel_radius*wheel_radius}" iyz="0.0"
-          izz="${wheel_mass / 12.0 * wheel_radius*wheel_radius}"/>
+          ixx="0.000270" ixy="0.0" ixz="0.0"
+          iyy="0.000270" iyz="0.0"
+          izz="0.000426"/>
       </inertial>
     </link>
