Commit message: Move ros2_control tags to separate xacro file

File: example_7/description/urdf/r6bot.urdf.xacro (robot description, xacro)
@@ -117,100 +117,6 @@
   </joint>
   <!-- ros2 control tag -->
-  <ros2_control name="r6bot" type="system">
-    <hardware>
-      <plugin>ros2_control_demo_example_7/RobotSystem</plugin>
-    </hardware>
-    <joint name="joint_1">
-      <command_interface name="position">
-        <param name="min">{-2*pi}</param>
-        <param name="max">{2*pi}</param>
-      </command_interface>
-      <command_interface name="velocity">
-        <param name="min">-3.15</param>
-        <param name="max">3.15</param>
-      </command_interface>
-      <state_interface name="position">
-        <param name="initial_value">0.0</param>
-      </state_interface>
-      <state_interface name="velocity"/>
-    </joint>
-    <joint name="joint_2">
-      <command_interface name="position">
-        <param name="min">{-2*pi}</param>
-        <param name="max">{2*pi}</param>
-      </command_interface>
-      <command_interface name="velocity">
-        <param name="min">-3.15</param>
-        <param name="max">3.15</param>
-      </command_interface>
-      <state_interface name="position">
-        <param name="initial_value">0.0</param>
-      </state_interface>
-      <state_interface name="velocity"/>
-    </joint>
-    <joint name="joint_3">
-      <command_interface name="position">
-        <param name="min">{-pi}</param>
-        <param name="max">{pi}</param>
-      </command_interface>
-      <command_interface name="velocity">
-        <param name="min">-3.15</param>
-        <param name="max">3.15</param>
-      </command_interface>
-      <state_interface name="position">
-        <param name="initial_value">0.0</param>
-      </state_interface>
-      <state_interface name="velocity"/>
-    </joint>
-    <joint name="joint_4">
-      <command_interface name="position">
-        <param name="min">{-2*pi}</param>
-        <param name="max">{2*pi}</param>
-      </command_interface>
-      <command_interface name="velocity">
-        <param name="min">-3.2</param>
-        <param name="max">3.2</param>
-      </command_interface>
-      <state_interface name="position">
-        <param name="initial_value">0.0</param>
-      </state_interface>
-      <state_interface name="velocity"/>
-    </joint>
-    <joint name="joint_5">
-      <command_interface name="position">
-        <param name="min">{-2*pi}</param>
-        <param name="max">{2*pi}</param>
-      </command_interface>
-      <command_interface name="velocity">
-        <param name="min">-3.2</param>
-        <param name="max">3.2</param>
-      </command_interface>
-      <state_interface name="position">
-        <param name="initial_value">0.0</param>
-      </state_interface>
-      <state_interface name="velocity"/>
-    </joint>
-    <joint name="joint_6">
-      <command_interface name="position">
-        <param name="min">{-2*pi}</param>
-        <param name="max">{2*pi}</param>
-      </command_interface>
-      <command_interface name="velocity">
-        <param name="min">-3.2</param>
-        <param name="max">3.2</param>
-      </command_interface>
-      <state_interface name="position">
-        <param name="initial_value">0.0</param>
-      </state_interface>
-      <state_interface name="velocity"/>
-    </joint>
-    <sensor name="tcp_fts_sensor">
-      <state_interface name="force.x"/>
-      <state_interface name="force.y"/>
-      <state_interface name="force.z"/>
-      <state_interface name="torque.x"/>
-      <state_interface name="torque.y"/>
-      <state_interface name="torque.z"/>
-    </sensor>
-  </ros2_control>
+  <!-- Import r6bot ros2_control description -->
+  <xacro:include filename="$(find ros2_control_demo_example_7)/ros2_control/r6bot.ros2_control.xacro" />
+  <xacro:r6bot_ros2_control name="r6bot"/>
 </robot>

Commit message: Move r6bot into description package

File: example_7/description/urdf/r6bot.urdf.xacro (robot description, xacro)
@@ -1,120 +1,9 @@
 <?xml version="1.0"?>
 <robot xmlns:xacro="http://wiki.ros.org/xacro" name="r6bot">
-  <!-- helper macro -->
-  <xacro:include filename="$(find ros2_control_demo_example_7)/urdf/inc/create_link.xacro"/>
+  <!-- Import r6bot macro -->
+  <xacro:include filename="$(find ros2_control_demo_description)/r6bot/urdf/r6bot_description.urdf.xacro"/>
   <!-- create link fixed to the "world" -->
   <link name="world"/>
-  <xacro:create_link
-      link_name="base_link"
-      xyz_offset="0 0 0"
-      rpy_offset="0 0 0"
-      mesh_package="ros2_control_demo_example_7"
-      mesh_name="link_0"
-  />
-  <xacro:create_link
-      link_name="link_1"
-      xyz_offset="0 0 0"
-      rpy_offset="0 0 0"
-      mesh_package="ros2_control_demo_example_7"
-      mesh_name="link_1"
-  />
-  <xacro:create_link
-      link_name="link_2"
-      xyz_offset="0 0 0"
-      rpy_offset="0 0 0"
-      mesh_package="ros2_control_demo_example_7"
-      mesh_name="link_2"
-  />
-  <xacro:create_link
-      link_name="link_3"
-      xyz_offset="0 0 0"
-      rpy_offset="0 0 0"
-      mesh_package="ros2_control_demo_example_7"
-      mesh_name="link_3"
-  />
-  <xacro:create_link
-      link_name="link_4"
-      xyz_offset="0 0 0"
-      rpy_offset="0 0 0"
-      mesh_package="ros2_control_demo_example_7"
-      mesh_name="link_4"
-  />
-  <xacro:create_link
-      link_name="link_5"
-      xyz_offset="0 0 0"
-      rpy_offset="0 0 0"
-      mesh_package="ros2_control_demo_example_7"
-      mesh_name="link_5"
-  />
-  <xacro:create_link
-      link_name="link_6"
-      xyz_offset="0 0 0"
-      rpy_offset="0 0 0"
-      mesh_package="ros2_control_demo_example_7"
-      mesh_name="link_6"
-  />
-  <link name="ft_frame"/>
-  <link name="tool0"/>
-  <!-- base_joint fixes base_link to the environment -->
-  <joint name="base_joint" type="fixed">
-    <parent link="world"/>
-    <child link="base_link"/>
-    <origin xyz="0 0 0" rpy="0 0 0"/>
-    <axis xyz="0 0 1"/>
-  </joint>
-  <!-- joints - main serial chain -->
-  <joint name="joint_1" type="revolute">
-    <parent link="base_link"/>
-    <child link="link_1"/>
-    <origin xyz="0 0 0.061584" rpy="0 0 0"/>
-    <axis xyz="0 0 1"/>
-    <limit effort="1000.0" lower="${-pi}" upper="${pi}" velocity="2.5"/>
-  </joint>
-  <joint name="joint_2" type="revolute">
-    <parent link="link_1"/>
-    <child link="link_2"/>
-    <origin xyz="-0.101717 0 0.182284" rpy="${-pi/2} -${pi/3} ${pi/2}"/>
-    <axis xyz="0 0 1"/>
-    <limit effort="1000.0" lower="${-pi}" upper="${pi}" velocity="2.5"/>
-  </joint>
-  <joint name="joint_3" type="revolute">
-    <parent link="link_2"/>
-    <child link="link_3"/>
-    <origin xyz="0.685682 0 0.041861" rpy="0 ${pi} ${pi+pi/2}"/>
-    <axis xyz="0 0 1"/>
-    <limit effort="1000.0" lower="${-pi}" upper="${pi}" velocity="2.5"/>
-  </joint>
-  <joint name="joint_4" type="revolute">
-    <parent link="link_3"/>
-    <child link="link_4"/>
-    <origin xyz="0.518777 0 0.067458" rpy="0 ${pi} ${pi+pi/6}"/>
-    <axis xyz="0 0 1"/>
-    <limit effort="1000.0" lower="${-pi}" upper="${pi}" velocity="2.5"/>
-  </joint>
-  <joint name="joint_5" type="revolute">
-    <parent link="link_4"/>
-    <child link="link_5"/>
-    <origin xyz="0.112654 0 0.110903" rpy="${pi/2} ${pi} ${pi/2}"/>
-    <axis xyz="0 0 1"/>
-    <limit effort="1000.0" lower="${-pi}" upper="${pi}" velocity="2.5"/>
-  </joint>
-  <joint name="joint_6" type="revolute">
-    <parent link="link_5"/>
-    <child link="link_6"/>
-    <origin xyz="-0.085976 0 0.133436" rpy="0 ${-pi/2} 0"/>
-    <axis xyz="0 0 1"/>
-    <limit effort="1000.0" lower="${-pi}" upper="${pi}" velocity="2.5"/>
-  </joint>
-  <joint name="joint-ft_frame" type="fixed">
-    <parent link="link_6"/>
-    <child link="ft_frame"/>
-    <origin xyz="0 0 0" rpy="0 0 0"/>
-  </joint>
-  <joint name="joint-tool" type="fixed">
-    <parent link="ft_frame"/>
-    <child link="tool0"/>
-    <origin xyz="0 0 .185" rpy="0 0 0"/>
-  </joint>
-  <!-- ros2 control tag -->
+  <xacro:r6bot_description/>
   <!-- Import r6bot ros2_control description -->
   <xacro:include filename="$(find ros2_control_demo_example_7)/ros2_control/r6bot.ros2_control.xacro" />
