Commit message: ackermann works with reference acceptance

File: example_11/description/urdf/carlikebot.urdf.xacro (robot description, xacro)
@@ -3,16 +3,9 @@
 <robot xmlns:xacro="http://www.ros.org/wiki/xacro" name="carlikebot_robot">
   <xacro:arg name="prefix" default="" />
-  <xacro:arg name="sim" default="true" />
+  <xacro:include filename="$(find ros2_control_demo_description)/carlikebot/urdf/carlikebot_description.urdf.xacro" />
   <!-- Import Rviz colors -->
-  <xacro:include filename="$(find ros2_control_demo_example_11)/urdf/carlikebot.materials.xacro" />
-  <!-- Import carlikebot description and ros2_control based on sim arg -->
-  <xacro:if value="$(arg sim)">
-    <xacro:include filename="$(find ros2_control_demo_example_11)/urdf/carlikebot_ackermann_description.urdf.xacro" />
-    <xacro:include filename="$(find ros2_control_demo_example_11)/ros2_control/carlikebot_ackermann.ros2_control.xacro" />
-  </xacro:if>
-  <xacro:unless value="$(arg sim)">
-    <xacro:include filename="$(find ros2_control_demo_example_11)/urdf/carlikebot_bicycle_description.urdf.xacro" />
-    <xacro:include filename="$(find ros2_control_demo_example_11)/ros2_control/carlikebot_bicycle.ros2_control.xacro" />
-  </xacro:unless>
+  <xacro:include filename="$(find ros2_control_demo_description)/carlikebot/urdf/carlikebot.materials.xacro" />
+  <!-- Import carlikebot ros2_control description -->
+  <xacro:include filename="$(find ros2_control_demo_example_11)/ros2_control/carlikebot.ros2_control.xacro" />
   <xacro:carlikebot prefix="$(arg prefix)" />
   <xacro:carlikebot_ros2_control

File: ros2_control_demo_description/carlikebot/urdf/carlikebot_description.urdf.xacro (robot description, xacro)
@@ -12,4 +12,5 @@
   <xacro:property name="wheel_len" value="0.045" />
   <xacro:property name="wheel_radius" value="0.05" />
+  <!-- <xacro:property name="wheeltrack" value="" -->
   <!-- Base Link -->
   <link name="${prefix}base_link" />
