Commit message: Add GenericSystem to GPIO example

File: example_10/description/ros2_control/rrbot.ros2_control.xacro (robot description, xacro)
@@ -1,12 +1,20 @@
 <?xml version="1.0"?>
 <robot xmlns:xacro="http://www.ros.org/wiki/xacro">
-  <xacro:macro name="rrbot_ros2_control" params="name prefix">
+  <xacro:macro name="rrbot_ros2_control" params="name prefix use_mock_hardware">
     <ros2_control name="${name}" type="system">
-      <hardware>
-        <plugin>ros2_control_demo_example_10/RRBotSystemWithGPIOHardware</plugin>
-        <param name="example_param_hw_start_duration_sec">0</param>
-        <param name="example_param_hw_stop_duration_sec">3.0</param>
-        <param name="example_param_hw_slowdown">100</param>
-      </hardware>
+      <xacro:unless value="${use_mock_hardware}">
+        <hardware>
+          <plugin>ros2_control_demo_example_10/RRBotSystemWithGPIOHardware</plugin>
+          <param name="example_param_hw_start_duration_sec">0</param>
+          <param name="example_param_hw_stop_duration_sec">3.0</param>
+          <param name="example_param_hw_slowdown">100</param>
+        </hardware>
+      </xacro:unless>
+      <xacro:if value="${use_mock_hardware}">
+        <hardware>
+          <plugin>mock_components/GenericSystem</plugin>
+          <param name="calculate_dynamics">true</param>
+        </hardware>
+      </xacro:if>
       <joint name="${prefix}joint1">
         <command_interface name="position">
@@ -32,5 +40,7 @@
       <gpio name="flange_vacuum">
         <command_interface name="vacuum"/>
-        <state_interface name="vacuum"/> <!-- Needed to know current state of the input -->
+        <state_interface name="vacuum">
+          <param name="initial_value">1.0</param>
+        </state_interface>
       </gpio>
     </ros2_control>

File: example_10/description/urdf/rrbot.urdf.xacro (robot description, xacro)
@@ -7,4 +7,5 @@
 <robot xmlns:xacro="http://www.ros.org/wiki/xacro" name="2dof_robot">
   <xacro:arg name="prefix" default="" />
+  <xacro:arg name="use_mock_hardware" default="false" />
   <!-- Import RRBot macro -->
   <xacro:include filename="$(find ros2_control_demo_description)/rrbot/urdf/rrbot_description.urdf.xacro" />
@@ -19,4 +20,4 @@
   </xacro:rrbot>
   <xacro:rrbot_ros2_control
-    name="RRBot" prefix="$(arg prefix)" />
+    name="RRBot" prefix="$(arg prefix)" use_mock_hardware="$(arg use_mock_hardware)"/>
 </robot>
