Commit message: Fix velocity limit

File: ros2_control_demo_description/carlikebot/urdf/carlikebot_description.urdf.xacro (robot description, xacro)
@@ -147,5 +147,5 @@
       <origin xyz="${wheelbase/2} 0 -${base_height/2}" rpy="0 0 ${PI/2}"/>
       <axis xyz="0 0 1"/>
-      <limit lower="-0.4" upper="0.4" effort="100.0" velocity="0.0"/>
+      <limit lower="-0.4" upper="0.4" effort="100.0" velocity="10.0"/>
       <dynamics damping="0.2"/>
     </joint>
@@ -179,5 +179,5 @@
       <origin xyz="${wheelbase/2} ${base_width/2} -${base_height/2}" rpy="0 0 ${PI/2}"/>
       <axis xyz="0 0 1"/>
-      <limit lower="-0.4" upper="0.4" effort="100.0" velocity="0.0"/>
+      <limit lower="-0.4" upper="0.4" effort="100.0" velocity="10.0"/>
       <dynamics damping="0.2"/>
       <mimic joint="${prefix}virtual_front_wheel_joint" multiplier="1.0" offset="0.0"/>
@@ -212,5 +212,5 @@
       <origin xyz="${wheelbase/2} -${base_width/2} -${base_height/2}" rpy="0 0 ${PI/2}"/>
       <axis xyz="0 0 1"/>
-      <limit lower="-0.4" upper="0.4" effort="100.0" velocity="0.0"/>
+      <limit lower="-0.4" upper="0.4" effort="100.0" velocity="10.0"/>
       <dynamics damping="0.2"/>
       <mimic joint="${prefix}virtual_front_wheel_joint" multiplier="1.0" offset="0.0"/>
