Commit message: Cleanup example 12

File: example_12/description/ros2_control/rrbot.ros2_control.xacro (robot description, xacro)
@@ -1,16 +1,11 @@
 <?xml version="1.0"?>
 <robot xmlns:xacro="http://www.ros.org/wiki/xacro">
-  <xacro:macro name="rrbot_ros2_control" params="name prefix use_gazebo_classic:=^|false">
+  <xacro:macro name="rrbot_ros2_control" params="name prefix">
     <ros2_control name="${name}" type="system">
       <hardware>
-        <xacro:if value="${use_gazebo_classic}">
-          <plugin>gazebo_ros2_control/GazeboSystem</plugin>
-        </xacro:if>
-        <xacro:unless value="${use_gazebo_classic}">
           <plugin>ros2_control_demo_example_12/RRBotSystemPositionOnlyHardware</plugin>
           <param name="example_param_hw_start_duration_sec">0</param>
           <param name="example_param_hw_stop_duration_sec">3.0</param>
           <param name="example_param_hw_slowdown">100</param>
-        </xacro:unless>
       </hardware>
       <joint name="${prefix}joint1">

File: example_12/description/urdf/rrbot.urdf.xacro (robot description, xacro)
@@ -7,5 +7,4 @@
 <robot xmlns:xacro="http://www.ros.org/wiki/xacro" name="2dof_robot">
   <xacro:arg name="prefix" default="" />
-  <xacro:arg name="use_gazebo_classic" default="false" />
   <!-- Import RRBot macro -->
   <xacro:include filename="$(find ros2_control_demo_description)/rrbot/urdf/rrbot_description.urdf.xacro" />
@@ -20,9 +19,4 @@
   </xacro:rrbot>
   <xacro:rrbot_ros2_control
-    name="RRBot" prefix="$(arg prefix)" use_gazebo_classic="$(arg use_gazebo_classic)"/>
-  <xacro:if value="$(arg use_gazebo_classic)">
-    <!-- Import Gazebo Classic definitions + plugin -->
-    <xacro:include filename="$(find ros2_control_demo_example_12)/gazebo/rrbot.gazebo.xacro" />
-    <xacro:rrbot_gazebo prefix="$(arg prefix)"/>
-  </xacro:if>
+    name="RRBot" prefix="$(arg prefix)"/>
 </robot>
