Commit message: Remove camera links etc

File: ros2_control_demo_description/r3bot/urdf/threedofbot_description.urdf.xacro (robot description, xacro)
@@ -141,68 +141,4 @@
         <link name="${prefix}tool_link">
         </link>
-        <joint name="${prefix}hokuyo_joint" type="fixed">
-          <axis xyz="0 1 0" />
-          <origin xyz="0 0 ${height4 - axel_offset/2}" rpy="0 0 0"/>
-          <parent link="${prefix}link3"/>
-          <child link="${prefix}hokuyo_link"/>
-        </joint>
-        <!-- Hokuyo Laser -->
-        <link name="${prefix}hokuyo_link">
-          <collision>
-            <origin xyz="0 0 0" rpy="0 0 0"/>
-            <geometry>
-              <box size="0.1 0.1 0.1"/>
-            </geometry>
-          </collision>
-          <visual>
-            <origin xyz="0 0 0" rpy="0 0 0"/>
-            <geometry>
-              <mesh filename="package://rrbot_description/meshes/hokuyo.dae"/>
-            </geometry>
-          </visual>
-          <inertial>
-            <mass value="1e-5" />
-            <origin xyz="0 0 0" rpy="0 0 0"/>
-            <inertia ixx="1e-6" ixy="0" ixz="0" iyy="1e-6" iyz="0" izz="1e-6" />
-          </inertial>
-        </link>
-        <joint name="${prefix}camera_joint" type="fixed">
-          <axis xyz="0 1 0" />
-          <origin xyz="${camera_link} 0 ${height4 - axel_offset*2}" rpy="0 0 0"/>
-          <parent link="${prefix}link2"/>
-          <child link="${prefix}camera_link"/>
-        </joint>
-        <!-- Camera -->
-        <link name="${prefix}camera_link">
-          <collision>
-            <origin xyz="0 0 0" rpy="0 0 0"/>
-            <geometry>
-              <box size="${camera_link} ${camera_link} ${camera_link}"/>
-            </geometry>
-          </collision>
-          <visual>
-            <origin xyz="0 0 0" rpy="0 0 0"/>
-            <geometry>
-              <box size="${camera_link} ${camera_link} ${camera_link}"/>
-            </geometry>
-            <material name="red"/>
-          </visual>
-          <inertial>
-            <mass value="1e-5" />
-            <origin xyz="0 0 0" rpy="0 0 0"/>
-            <inertia ixx="1e-6" ixy="0" ixz="0" iyy="1e-6" iyz="0" izz="1e-6" />
-          </inertial>
-        </link>
-        <!-- generate an optical frame http://www.ros.org/reps/rep-0103.html#suffix-frames
-        so that ros and opencv can operate on the camera frame correctly -->
-        <joint name="${prefix}camera_optical_joint" type="fixed">
-          <!-- these values have to be these values otherwise the gazebo camera image
-          won't be aligned properly with the frame it is supposedly originating from -->
-          <origin xyz="0 0 0" rpy="${-pi/2} 0 ${-pi/2}"/>
-          <parent link="${prefix}camera_link"/>
-          <child link="${prefix}camera_link_optical"/>
-        </joint>
-        <link name="${prefix}camera_link_optical">
-        </link>
   </xacro:macro>
 </robot>
