Commit message: Add limits to the continuous joints

File: ros2_control_demo_description/diffbot/urdf/diffbot_description.urdf.xacro (robot description, xacro)
@@ -44,4 +44,5 @@
       <axis xyz="0 1 0"/>
       <dynamics damping="0.2"/>
+      <limit effort="100" velocity="1.0"/>
     </joint>
     <!-- left wheel Link -->
@@ -75,4 +76,5 @@
       <axis xyz="0 1 0"/>
       <dynamics damping="0.2"/>
+      <limit effort="100" velocity="1.0"/>
     </joint>
     <!-- right wheel Link -->

File: ros2_control_demo_description/rrbot/urdf/rrbot_description.urdf.xacro (robot description, xacro)
@@ -44,4 +44,5 @@
     <axis xyz="0 1 0"/>
     <dynamics damping="0.7"/>
+    <limit effort="100" velocity="1.0"/>
   </joint>
   <!-- Middle Link -->
@@ -75,4 +76,5 @@
     <axis xyz="0 1 0"/>
     <dynamics damping="0.7"/>
+    <limit effort="100" velocity="1.0"/>
   </joint>
   <!-- Top Link -->

Commit message: Added example_17: chained controllers for diff drive using effort interface and Gazebo.
Signed-off-by: Martin Pecka <peckama2@fel.cvut.cz>

File: ros2_control_demo_description/diffbot/urdf/diffbot_description.urdf.xacro (robot description, xacro)
@@ -44,5 +44,5 @@
       <axis xyz="0 1 0"/>
       <dynamics damping="0.2"/>
-      <limit effort="100" velocity="1.0"/>
+      <limit effort="100" velocity="60.0"/>
     </joint>
     <!-- left wheel Link -->
@@ -76,5 +76,5 @@
       <axis xyz="0 1 0"/>
       <dynamics damping="0.2"/>
-      <limit effort="100" velocity="1.0"/>
+      <limit effort="100" velocity="60.0"/>
     </joint>
     <!-- right wheel Link -->
