Commit message: Switch from gazebo classic to gazebo

File: example_9/description/gazebo/rrbot.gazebo.xacro (robot description, xacro)
@@ -8,5 +8,5 @@
     <!-- ros_control plugin -->
     <gazebo>
-      <plugin filename="libgazebo_ros2_control.so" name="gazebo_ros2_control">
+      <plugin filename="gz_ros2_control-system" name="gz_ros2_control::GazeboSimROS2ControlPlugin">
         <parameters>$(find ros2_control_demo_example_9)/config/rrbot_controllers.yaml</parameters>
       </plugin>

File: example_9/description/ros2_control/rrbot.ros2_control.xacro (robot description, xacro)
@@ -1,11 +1,11 @@
 <?xml version="1.0"?>
 <robot xmlns:xacro="http://www.ros.org/wiki/xacro">
-  <xacro:macro name="rrbot_ros2_control" params="name prefix use_gazebo_classic:=^|false">
+  <xacro:macro name="rrbot_ros2_control" params="name prefix use_gazebo:=^|false">
     <ros2_control name="${name}" type="system">
       <hardware>
-        <xacro:if value="${use_gazebo_classic}">
-          <plugin>gazebo_ros2_control/GazeboSystem</plugin>
+        <xacro:if value="${use_gazebo}">
+          <plugin>gz_ros2_control/GazeboSimSystem</plugin>
         </xacro:if>
-        <xacro:unless value="${use_gazebo_classic}">
+        <xacro:unless value="${use_gazebo}">
           <plugin>ros2_control_demo_example_9/RRBotSystemPositionOnlyHardware</plugin>
           <param name="example_param_hw_start_duration_sec">0</param>

File: example_9/description/urdf/rrbot.urdf.xacro (robot description, xacro)
@@ -7,5 +7,5 @@
 <robot xmlns:xacro="http://www.ros.org/wiki/xacro" name="2dof_robot">
   <xacro:arg name="prefix" default="" />
-  <xacro:arg name="use_gazebo_classic" default="false" />
+  <xacro:arg name="use_gazebo" default="false" />
   <!-- Import RRBot macro -->
   <xacro:include filename="$(find ros2_control_demo_description)/rrbot/urdf/rrbot_description.urdf.xacro" />
@@ -20,6 +20,6 @@
   </xacro:rrbot>
   <xacro:rrbot_ros2_control
-    name="RRBot" prefix="$(arg prefix)" use_gazebo_classic="$(arg use_gazebo_classic)"/>
-  <xacro:if value="$(arg use_gazebo_classic)">
+    name="RRBot" prefix="$(arg prefix)" use_gazebo="$(arg use_gazebo)"/>
+  <xacro:if value="$(arg use_gazebo)">
     <!-- Import Gazebo Classic definitions + plugin -->
     <xacro:include filename="$(find ros2_control_demo_example_9)/gazebo/rrbot.gazebo.xacro" />

Commit message: Working version.

File: example_9/description/gazebo/rrbot.gazebo.xacro (robot description, xacro)
@@ -6,8 +6,11 @@
 <robot xmlns:xacro="http://ros.org/wiki/xacro">
   <xacro:macro name="rrbot_gazebo" params="prefix">
-    <!-- ros_control plugin -->
+    <!-- ros2_control GZ Sim plugin -->
+    <gazebo reference="world">
+    </gazebo>
     <gazebo>
-      <plugin filename="libgazebo_ros2_control.so" name="gazebo_ros2_control">
+      <plugin filename="gz_ros2_control-system" name="gz_ros2_control::GazeboSimROS2ControlPlugin">
         <parameters>$(find ros2_control_demo_example_9)/config/rrbot_controllers.yaml</parameters>
+        <controller_manager_node_name>${prefix}controller_manager</controller_manager_node_name>
       </plugin>
     </gazebo>

File: example_9/description/ros2_control/rrbot.ros2_control.xacro (robot description, xacro)
@@ -1,11 +1,11 @@
 <?xml version="1.0"?>
 <robot xmlns:xacro="http://www.ros.org/wiki/xacro">
-  <xacro:macro name="rrbot_ros2_control" params="name prefix use_gazebo_classic:=^|false">
+  <xacro:macro name="rrbot_ros2_control" params="name prefix use_gazebo_sim:=^|false">
     <ros2_control name="${name}" type="system">
       <hardware>
-        <xacro:if value="${use_gazebo_classic}">
-          <plugin>gazebo_ros2_control/GazeboSystem</plugin>
+        <xacro:if value="${use_gazebo_sim}">
+          <plugin>gz_ros2_control/GazeboSimSystem</plugin>
         </xacro:if>
-        <xacro:unless value="${use_gazebo_classic}">
+        <xacro:unless value="${use_gazebo_sim}">
           <plugin>ros2_control_demo_example_9/RRBotSystemPositionOnlyHardware</plugin>
           <param name="example_param_hw_start_duration_sec">0</param>

File: example_9/description/urdf/rrbot.urdf.xacro (robot description, xacro)
@@ -7,5 +7,5 @@
 <robot xmlns:xacro="http://www.ros.org/wiki/xacro" name="2dof_robot">
   <xacro:arg name="prefix" default="" />
-  <xacro:arg name="use_gazebo_classic" default="false" />
+  <xacro:arg name="use_gazebo_sim" default="false" />
   <!-- Import RRBot macro -->
   <xacro:include filename="$(find ros2_control_demo_description)/rrbot/urdf/rrbot_description.urdf.xacro" />
@@ -20,6 +20,6 @@
   </xacro:rrbot>
   <xacro:rrbot_ros2_control
-    name="RRBot" prefix="$(arg prefix)" use_gazebo_classic="$(arg use_gazebo_classic)"/>
-  <xacro:if value="$(arg use_gazebo_classic)">
+    name="RRBot" prefix="$(arg prefix)" use_gazebo_sim="$(arg use_gazebo_sim)"/>
+  <xacro:if value="$(arg use_gazebo_sim)">
     <!-- Import Gazebo Classic definitions + plugin -->
     <xacro:include filename="$(find ros2_control_demo_example_9)/gazebo/rrbot.gazebo.xacro" />

Commit message: Add gazebo bridge node

File: example_9/description/gazebo/rrbot.gazebo.xacro (robot description, xacro)
@@ -14,5 +14,10 @@
     <!-- Link1 -->
     <gazebo reference="${prefix}base_link">
-      <material>Gazebo/Orange</material>
+      <material>
+        <script>
+          <uri>file://media/materials/scripts/gazebo.material</uri>
+          <name>Gazebo/Orange</name>
+        </script>
+      </material>
     </gazebo>
     <!-- Link2 -->
@@ -20,5 +25,10 @@
       <mu1>0.2</mu1>
       <mu2>0.2</mu2>
-      <material>Gazebo/Yellow</material>
+      <material>
+        <script>
+          <uri>file://media/materials/scripts/gazebo.material</uri>
+          <name>Gazebo/Yellow</name>
+        </script>
+      </material>
     </gazebo>
     <!-- Link3 -->
@@ -26,5 +36,10 @@
       <mu1>0.2</mu1>
       <mu2>0.2</mu2>
-      <material>Gazebo/Orange</material>
+      <material>
+        <script>
+          <uri>file://media/materials/scripts/gazebo.material</uri>
+          <name>Gazebo/Yellow</name>
+        </script>
+      </material>
     </gazebo>
   </xacro:macro>

Commit message: [example_9] Switch to gz_ros2_control (backport #482) (#749)
* [example_9] Switch to gz_ros2_control (#482)

* Switch from gazebo classic to gazebo

* update docs

* Use gz_ros2_control in semi-binary builds

* rm dependency conditional

Co-authored-by: Dr. Denis <denis@stogl.de>

* Remove gazebo classic from repos file

* Add gazebo bridge node and fix some warnings (#755) (#757)

(cherry picked from commit 25879705bcb6135632242df547d266be45902fc4)

Co-authored-by: Julia Jia <juliajster@gmail.com>

---------

Co-authored-by: Christoph Fröhlich <christophfroehlich@users.noreply.github.com>
Co-authored-by: Dr. Denis <denis@stogl.de>
Co-authored-by: Christoph Froehlich <christoph.froehlich@ait.ac.at>
Co-authored-by: mergify[bot] <37929162+mergify[bot]@users.noreply.github.com>
Co-authored-by: Julia Jia <juliajster@gmail.com>

File: example_9/description/gazebo/rrbot.gazebo.xacro (robot description, xacro)
@@ -8,5 +8,5 @@
     <!-- ros_control plugin -->
     <gazebo>
-      <plugin filename="libgazebo_ros2_control.so" name="gazebo_ros2_control">
+      <plugin filename="gz_ros2_control-system" name="gz_ros2_control::GazeboSimROS2ControlPlugin">
         <parameters>$(find ros2_control_demo_example_9)/config/rrbot_controllers.yaml</parameters>
       </plugin>
@@ -14,5 +14,10 @@
     <!-- Link1 -->
     <gazebo reference="${prefix}base_link">
-      <material>Gazebo/Orange</material>
+      <material>
+        <script>
+          <uri>file://media/materials/scripts/gazebo.material</uri>
+          <name>Gazebo/Orange</name>
+        </script>
+      </material>
     </gazebo>
     <!-- Link2 -->
@@ -20,5 +25,10 @@
       <mu1>0.2</mu1>
       <mu2>0.2</mu2>
-      <material>Gazebo/Yellow</material>
+      <material>
+        <script>
+          <uri>file://media/materials/scripts/gazebo.material</uri>
+          <name>Gazebo/Yellow</name>
+        </script>
+      </material>
     </gazebo>
     <!-- Link3 -->
@@ -26,5 +36,10 @@
       <mu1>0.2</mu1>
       <mu2>0.2</mu2>
-      <material>Gazebo/Orange</material>
+      <material>
+        <script>
+          <uri>file://media/materials/scripts/gazebo.material</uri>
+          <name>Gazebo/Yellow</name>
+        </script>
+      </material>
     </gazebo>
   </xacro:macro>
