Commit message: Switch order of hardware components

File: example_14/description/ros2_control/rrbot_modular_actuators_without_feedback_sensors_for_position_feedback.ros2_control.xacro (robot description, xacro)
@@ -5,34 +5,10 @@
     <!-- NOTE generally is the order of hardware definition not relevant. But in this case the
     sensors are listening on sockets to which the actuators are connecting. Therefore, the sensors
-    has to be initialized and started first. -->
-    <ros2_control name="RRBotModularPositionSensorJoint1" type="sensor">
-      <hardware>
-        <plugin>ros2_control_demo_example_14/RRBotSensorPositionFeedback</plugin>
-        <param name="example_param_hw_start_duration_sec">1.0</param>
-        <param name="example_param_hw_stop_duration_sec">2.0</param>
-        <param name="example_param_hw_slowdown">${slowdown}</param>
-        <param name="example_param_socket_port">23286</param>
-      </hardware>
-      <joint name="joint1">
-        <state_interface name="position"/>
-      </joint>
-    </ros2_control>
-    <ros2_control name="RRBotModularPositionSensorJoint2" type="sensor">
-      <hardware>
-        <plugin>ros2_control_demo_example_14/RRBotSensorPositionFeedback</plugin>
-        <param name="example_param_hw_start_duration_sec">1.0</param>
-        <param name="example_param_hw_stop_duration_sec">2.0</param>
-        <param name="example_param_hw_slowdown">${slowdown}</param>
-        <param name="example_param_socket_port">23287</param>
-      </hardware>
-      <joint name="joint2">
-        <state_interface name="position"/>
-      </joint>
-    </ros2_control>
+    has to be initialized and configured first. Note: configuration will be done in reverse order. -->
     <ros2_control name="RRBotModularJoint1" type="actuator">
       <hardware>
         <plugin>ros2_control_demo_example_14/RRBotActuatorWithoutFeedback</plugin>
         <param name="example_param_hw_start_duration_sec">2.0</param>
-        <param name="example_param_hw_stop_duration_sec">3.0</param>
+        <param name="example_param_hw_stop_duration_sec">1.0</param>
         <param name="example_param_socket_port">23286</param>
       </hardware>
@@ -48,5 +24,5 @@
         <plugin>ros2_control_demo_example_14/RRBotActuatorWithoutFeedback</plugin>
         <param name="example_param_hw_start_duration_sec">2.0</param>
-        <param name="example_param_hw_stop_duration_sec">3.0</param>
+        <param name="example_param_hw_stop_duration_sec">1.0</param>
         <param name="example_param_socket_port">23287</param>
       </hardware>
@@ -57,5 +33,29 @@
         </command_interface>
       </joint>
-      </ros2_control>
+    </ros2_control>
+    <ros2_control name="RRBotModularPositionSensorJoint1" type="sensor">
+      <hardware>
+        <plugin>ros2_control_demo_example_14/RRBotSensorPositionFeedback</plugin>
+        <param name="example_param_hw_start_duration_sec">1.0</param>
+        <param name="example_param_hw_stop_duration_sec">0.0</param>
+        <param name="example_param_hw_slowdown">${slowdown}</param>
+        <param name="example_param_socket_port">23286</param>
+      </hardware>
+      <joint name="joint1">
+        <state_interface name="position"/>
+      </joint>
+    </ros2_control>
+    <ros2_control name="RRBotModularPositionSensorJoint2" type="sensor">
+      <hardware>
+        <plugin>ros2_control_demo_example_14/RRBotSensorPositionFeedback</plugin>
+        <param name="example_param_hw_start_duration_sec">1.0</param>
+        <param name="example_param_hw_stop_duration_sec">0.0</param>
+        <param name="example_param_hw_slowdown">${slowdown}</param>
+        <param name="example_param_socket_port">23287</param>
+      </hardware>
+      <joint name="joint2">
+        <state_interface name="position"/>
+      </joint>
+    </ros2_control>
   </xacro:macro>
 </robot>

Commit message: Fix thread stopping of example_14 (#850)
(cherry picked from commit 65a8fbc6d76b06ecd19df1ce230cc00379cab72f)

# Conflicts:
#	example_14/description/ros2_control/rrbot_modular_actuators_without_feedback_sensors_for_position_feedback.ros2_control.xacro
#	example_14/hardware/include/ros2_control_demo_example_14/rrbot_sensor_for_position_feedback.hpp
#	example_14/hardware/rrbot_actuator_without_feedback.cpp
#	example_14/hardware/rrbot_sensor_for_position_feedback.cpp

File: example_14/description/ros2_control/rrbot_modular_actuators_without_feedback_sensors_for_position_feedback.ros2_control.xacro (robot description, xacro)
@@ -4,4 +4,5 @@
     params="name prefix use_sim:=^|false slowdown:=2.0">
     <!-- NOTE generally is the order of hardware definition not relevant. But in this case the
+<<<<<<< HEAD
     sensors are listening on socket to which the actuators are connecting. Therefore, the sensors
     has to be initialized and started first. -->
@@ -30,9 +31,13 @@
       </joint>
       </ros2_control>
+=======
+    sensors are listening on sockets to which the actuators are connecting. Therefore, the sensors
+    has to be initialized and configured first. Configuration will be done in reverse order. -->
+>>>>>>> 65a8fbc (Fix thread stopping of example_14 (#850))
     <ros2_control name="RRBotModularJoint1" type="actuator">
       <hardware>
         <plugin>ros2_control_demo_example_14/RRBotActuatorWithoutFeedback</plugin>
         <param name="example_param_hw_start_duration_sec">2.0</param>
-        <param name="example_param_hw_stop_duration_sec">3.0</param>
+        <param name="example_param_hw_stop_duration_sec">1.0</param>
         <param name="example_param_socket_port">23286</param>
       </hardware>
@@ -48,5 +53,5 @@
         <plugin>ros2_control_demo_example_14/RRBotActuatorWithoutFeedback</plugin>
         <param name="example_param_hw_start_duration_sec">2.0</param>
-        <param name="example_param_hw_stop_duration_sec">3.0</param>
+        <param name="example_param_hw_stop_duration_sec">1.0</param>
         <param name="example_param_socket_port">23287</param>
       </hardware>
@@ -57,5 +62,29 @@
         </command_interface>
       </joint>
-      </ros2_control>
+    </ros2_control>
+    <ros2_control name="RRBotModularPositionSensorJoint1" type="sensor">
+      <hardware>
+        <plugin>ros2_control_demo_example_14/RRBotSensorPositionFeedback</plugin>
+        <param name="example_param_hw_start_duration_sec">1.0</param>
+        <param name="example_param_hw_stop_duration_sec">0.0</param>
+        <param name="example_param_hw_slowdown">${slowdown}</param>
+        <param name="example_param_socket_port">23286</param>
+      </hardware>
+      <joint name="joint1">
+        <state_interface name="position"/>
+      </joint>
+    </ros2_control>
+    <ros2_control name="RRBotModularPositionSensorJoint2" type="sensor">
+      <hardware>
+        <plugin>ros2_control_demo_example_14/RRBotSensorPositionFeedback</plugin>
+        <param name="example_param_hw_start_duration_sec">1.0</param>
+        <param name="example_param_hw_stop_duration_sec">0.0</param>
+        <param name="example_param_hw_slowdown">${slowdown}</param>
+        <param name="example_param_socket_port">23287</param>
+      </hardware>
+      <joint name="joint2">
+        <state_interface name="position"/>
+      </joint>
+    </ros2_control>
   </xacro:macro>
 </robot>

Commit message: Fix thread stopping of example_14 (#850)

File: example_14/description/ros2_control/rrbot_modular_actuators_without_feedback_sensors_for_position_feedback.ros2_control.xacro (robot description, xacro)
@@ -5,34 +5,10 @@
     <!-- NOTE generally is the order of hardware definition not relevant. But in this case the
     sensors are listening on sockets to which the actuators are connecting. Therefore, the sensors
-    has to be initialized and started first. -->
-    <ros2_control name="RRBotModularPositionSensorJoint1" type="sensor">
-      <hardware>
-        <plugin>ros2_control_demo_example_14/RRBotSensorPositionFeedback</plugin>
-        <param name="example_param_hw_start_duration_sec">1.0</param>
-        <param name="example_param_hw_stop_duration_sec">2.0</param>
-        <param name="example_param_hw_slowdown">${slowdown}</param>
-        <param name="example_param_socket_port">23286</param>
-      </hardware>
-      <joint name="joint1">
-        <state_interface name="position"/>
-      </joint>
-    </ros2_control>
-    <ros2_control name="RRBotModularPositionSensorJoint2" type="sensor">
-      <hardware>
-        <plugin>ros2_control_demo_example_14/RRBotSensorPositionFeedback</plugin>
-        <param name="example_param_hw_start_duration_sec">1.0</param>
-        <param name="example_param_hw_stop_duration_sec">2.0</param>
-        <param name="example_param_hw_slowdown">${slowdown}</param>
-        <param name="example_param_socket_port">23287</param>
-      </hardware>
-      <joint name="joint2">
-        <state_interface name="position"/>
-      </joint>
-    </ros2_control>
+    has to be initialized and configured first. Configuration will be done in reverse order. -->
     <ros2_control name="RRBotModularJoint1" type="actuator">
       <hardware>
         <plugin>ros2_control_demo_example_14/RRBotActuatorWithoutFeedback</plugin>
         <param name="example_param_hw_start_duration_sec">2.0</param>
-        <param name="example_param_hw_stop_duration_sec">3.0</param>
+        <param name="example_param_hw_stop_duration_sec">1.0</param>
         <param name="example_param_socket_port">23286</param>
       </hardware>
@@ -48,5 +24,5 @@
         <plugin>ros2_control_demo_example_14/RRBotActuatorWithoutFeedback</plugin>
         <param name="example_param_hw_start_duration_sec">2.0</param>
-        <param name="example_param_hw_stop_duration_sec">3.0</param>
+        <param name="example_param_hw_stop_duration_sec">1.0</param>
         <param name="example_param_socket_port">23287</param>
       </hardware>
@@ -57,5 +33,29 @@
         </command_interface>
       </joint>
-      </ros2_control>
+    </ros2_control>
+    <ros2_control name="RRBotModularPositionSensorJoint1" type="sensor">
+      <hardware>
+        <plugin>ros2_control_demo_example_14/RRBotSensorPositionFeedback</plugin>
+        <param name="example_param_hw_start_duration_sec">1.0</param>
+        <param name="example_param_hw_stop_duration_sec">0.0</param>
+        <param name="example_param_hw_slowdown">${slowdown}</param>
+        <param name="example_param_socket_port">23286</param>
+      </hardware>
+      <joint name="joint1">
+        <state_interface name="position"/>
+      </joint>
+    </ros2_control>
+    <ros2_control name="RRBotModularPositionSensorJoint2" type="sensor">
+      <hardware>
+        <plugin>ros2_control_demo_example_14/RRBotSensorPositionFeedback</plugin>
+        <param name="example_param_hw_start_duration_sec">1.0</param>
+        <param name="example_param_hw_stop_duration_sec">0.0</param>
+        <param name="example_param_hw_slowdown">${slowdown}</param>
+        <param name="example_param_socket_port">23287</param>
+      </hardware>
+      <joint name="joint2">
+        <state_interface name="position"/>
+      </joint>
+    </ros2_control>
   </xacro:macro>
 </robot>

Commit message: Fix merge conflicts

File: example_14/description/ros2_control/rrbot_modular_actuators_without_feedback_sensors_for_position_feedback.ros2_control.xacro (robot description, xacro)
@@ -4,35 +4,6 @@
     params="name prefix use_sim:=^|false slowdown:=2.0">
     <!-- NOTE generally is the order of hardware definition not relevant. But in this case the
-<<<<<<< HEAD
-    sensors are listening on socket to which the actuators are connecting. Therefore, the sensors
-    has to be initialized and started first. -->
-    <ros2_control name="RRBotModularPositionSensorJoint1" type="sensor">
-      <hardware>
-        <plugin>ros2_control_demo_example_14/RRBotSensorPositionFeedback</plugin>
-        <param name="example_param_hw_start_duration_sec">1.0</param>
-        <param name="example_param_hw_stop_duration_sec">2.0</param>
-        <param name="example_param_hw_slowdown">${slowdown}</param>
-        <param name="example_param_socket_port">23286</param>
-      </hardware>
-      <joint name="joint1">
-        <state_interface name="position"/>
-      </joint>
-    </ros2_control>
-    <ros2_control name="RRBotModularPositionSensorJoint2" type="sensor">
-      <hardware>
-        <plugin>ros2_control_demo_example_14/RRBotSensorPositionFeedback</plugin>
-        <param name="example_param_hw_start_duration_sec">1.0</param>
-        <param name="example_param_hw_stop_duration_sec">2.0</param>
-        <param name="example_param_hw_slowdown">${slowdown}</param>
-        <param name="example_param_socket_port">23287</param>
-      </hardware>
-      <joint name="joint2">
-        <state_interface name="position"/>
-      </joint>
-      </ros2_control>
-=======
     sensors are listening on sockets to which the actuators are connecting. Therefore, the sensors
     has to be initialized and configured first. Configuration will be done in reverse order. -->
->>>>>>> 65a8fbc (Fix thread stopping of example_14 (#850))
     <ros2_control name="RRBotModularJoint1" type="actuator">
       <hardware>

Commit message: Fix thread stopping of example_14 (backport #850) (#851)

File: example_14/description/ros2_control/rrbot_modular_actuators_without_feedback_sensors_for_position_feedback.ros2_control.xacro (robot description, xacro)
@@ -4,35 +4,11 @@
     params="name prefix use_sim:=^|false slowdown:=2.0">
     <!-- NOTE generally is the order of hardware definition not relevant. But in this case the
-    sensors are listening on socket to which the actuators are connecting. Therefore, the sensors
-    has to be initialized and started first. -->
-    <ros2_control name="RRBotModularPositionSensorJoint1" type="sensor">
-      <hardware>
-        <plugin>ros2_control_demo_example_14/RRBotSensorPositionFeedback</plugin>
-        <param name="example_param_hw_start_duration_sec">1.0</param>
-        <param name="example_param_hw_stop_duration_sec">2.0</param>
-        <param name="example_param_hw_slowdown">${slowdown}</param>
-        <param name="example_param_socket_port">23286</param>
-      </hardware>
-      <joint name="joint1">
-        <state_interface name="position"/>
-      </joint>
-    </ros2_control>
-    <ros2_control name="RRBotModularPositionSensorJoint2" type="sensor">
-      <hardware>
-        <plugin>ros2_control_demo_example_14/RRBotSensorPositionFeedback</plugin>
-        <param name="example_param_hw_start_duration_sec">1.0</param>
-        <param name="example_param_hw_stop_duration_sec">2.0</param>
-        <param name="example_param_hw_slowdown">${slowdown}</param>
-        <param name="example_param_socket_port">23287</param>
-      </hardware>
-      <joint name="joint2">
-        <state_interface name="position"/>
-      </joint>
-      </ros2_control>
+    sensors are listening on sockets to which the actuators are connecting. Therefore, the sensors
+    has to be initialized and configured first. Configuration will be done in reverse order. -->
     <ros2_control name="RRBotModularJoint1" type="actuator">
       <hardware>
         <plugin>ros2_control_demo_example_14/RRBotActuatorWithoutFeedback</plugin>
         <param name="example_param_hw_start_duration_sec">2.0</param>
-        <param name="example_param_hw_stop_duration_sec">3.0</param>
+        <param name="example_param_hw_stop_duration_sec">1.0</param>
         <param name="example_param_socket_port">23286</param>
       </hardware>
@@ -48,5 +24,5 @@
         <plugin>ros2_control_demo_example_14/RRBotActuatorWithoutFeedback</plugin>
         <param name="example_param_hw_start_duration_sec">2.0</param>
-        <param name="example_param_hw_stop_duration_sec">3.0</param>
+        <param name="example_param_hw_stop_duration_sec">1.0</param>
         <param name="example_param_socket_port">23287</param>
       </hardware>
@@ -57,5 +33,29 @@
         </command_interface>
       </joint>
-      </ros2_control>
+    </ros2_control>
+    <ros2_control name="RRBotModularPositionSensorJoint1" type="sensor">
+      <hardware>
+        <plugin>ros2_control_demo_example_14/RRBotSensorPositionFeedback</plugin>
+        <param name="example_param_hw_start_duration_sec">1.0</param>
+        <param name="example_param_hw_stop_duration_sec">0.0</param>
+        <param name="example_param_hw_slowdown">${slowdown}</param>
+        <param name="example_param_socket_port">23286</param>
+      </hardware>
+      <joint name="joint1">
+        <state_interface name="position"/>
+      </joint>
+    </ros2_control>
+    <ros2_control name="RRBotModularPositionSensorJoint2" type="sensor">
+      <hardware>
+        <plugin>ros2_control_demo_example_14/RRBotSensorPositionFeedback</plugin>
+        <param name="example_param_hw_start_duration_sec">1.0</param>
+        <param name="example_param_hw_stop_duration_sec">0.0</param>
+        <param name="example_param_hw_slowdown">${slowdown}</param>
+        <param name="example_param_socket_port">23287</param>
+      </hardware>
+      <joint name="joint2">
+        <state_interface name="position"/>
+      </joint>
+    </ros2_control>
   </xacro:macro>
 </robot>
