Commit message: Enabling rolling-semi-binary-build and switch to use onnxruntime_vendor

File: example_18/description/ros2_control/open_duck_mini.ros2_control.xacro (robot description, xacro)
@@ -3,7 +3,7 @@
   <!-- 14 DoF: left leg (0-4), head (5-8), right leg (9-13). Ref: example_config.json -->
   <xacro:macro name="open_duck_mini_mujoco_ros2_control" params="name prefix">
-    <xacro:open_duck_mini_ros2_control name="${name}" prefix="${prefix}" use_mock_hardware="false"/>
+    <xacro:open_duck_mini_ros2_control name="${name}" prefix="${prefix}" use_mock_hardware="false" headless="false"/>
   </xacro:macro>
-  <xacro:macro name="open_duck_mini_ros2_control" params="name prefix use_mock_hardware:=^|false">
+  <xacro:macro name="open_duck_mini_ros2_control" params="name prefix use_mock_hardware:=^|false headless:=^|false">
     <ros2_control name="${name}" type="system">
       <xacro:unless value="${use_mock_hardware}">
@@ -14,4 +14,5 @@
           <!-- External PID disabled: MuJoCo built-in actuators used -->
           <param name="override_start_position_file">$(find ros2_control_demo_example_18)/description/mujoco/start_positions.xml</param>
+          <param name="headless">${headless}</param>
         </hardware>
       </xacro:unless>

File: example_18/description/urdf/open_duck_mini.urdf.xacro (robot description, xacro)
@@ -9,4 +9,5 @@
   <xacro:arg name="prefix" default="" />
   <xacro:arg name="use_mock_hardware" default="false" />
+  <xacro:arg name="headless" default="false" />
   <!-- Include the base URDF description -->
   <!-- Note: xacro will process the URDF file and merge its content -->
@@ -15,4 +16,4 @@
   <xacro:include filename="$(find ros2_control_demo_example_18)/description/ros2_control/open_duck_mini.ros2_control.xacro" />
   <xacro:open_duck_mini_ros2_control
-    name="OpenDuckMini" prefix="$(arg prefix)" use_mock_hardware="$(arg use_mock_hardware)"/>
+    name="OpenDuckMini" prefix="$(arg prefix)" use_mock_hardware="$(arg use_mock_hardware)" headless="$(arg headless)"/>
 </robot>
