Commit message: Move open duck mini assets to ros2_control_demo_description package

File: ros2_control_demo_description/openduckmini/mujoco/robot.urdf (robot description, URDF)
Before this commit: robot open-duck-mini, 16 links, 15 joints
Links:
- link head_pitch_link: geometry visual mesh filename=package://ros2_control_demo_description/openduckmini/assets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
- link head_roll_link: geometry visual mesh filename=package://ros2_control_demo_description/openduckmini/assets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; visual mesh filename=package://ros2_control_demo_description/openduckmini/assets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
- link head_yaw_link: geometry visual mesh filename=package://ros2_control_demo_description/openduckmini/assets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
- link left_ankle_link: geometry visual mesh filename=package://ros2_control_demo_description/openduckmini/assets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; visual mesh filename=package://ros2_control_demo_description/openduckmini/assets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
- link left_hip_pitch_link: geometry visual mesh filename=package://ros2_control_demo_description/openduckmini/assets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; visual mesh filename=package://ros2_control_demo_description/openduckmini/assets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
- link left_hip_roll_link: geometry visual mesh filename=package://ros2_control_demo_description/openduckmini/assets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
- link left_hip_yaw_link: geometry visual mesh filename=package://ros2_control_demo_description/openduckmini/assets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; visual mesh filename=package://ros2_control_demo_description/openduckmini/assets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
- link left_knee_link: geometry visual mesh filename=package://ros2_control_demo_description/openduckmini/assets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; visual mesh filename=package://ros2_control_demo_description/openduckmini/assets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
- link neck_pitch_link: geometry visual mesh filename=package://ros2_control_demo_description/openduckmini/assets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; visual mesh filename=package://ros2_control_demo_description/openduckmini/assets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
- link right_ankle_link: geometry visual mesh filename=package://ros2_control_demo_description/openduckmini/assets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; visual mesh filename=package://ros2_control_demo_description/openduckmini/assets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
- link right_hip_pitch_link: geometry visual mesh filename=package://ros2_control_demo_description/openduckmini/assets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; visual mesh filename=package://ros2_control_demo_description/openduckmini/assets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
- link right_hip_roll_link: geometry visual mesh filename=package://ros2_control_demo_description/openduckmini/assets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
- link right_hip_yaw_link: geometry visual mesh filename=package://ros2_control_demo_description/openduckmini/assets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; visual mesh filename=package://ros2_control_demo_description/openduckmini/assets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
- link right_knee_link: geometry visual mesh filename=package://ros2_control_demo_description/openduckmini/assets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; visual mesh filename=package://ros2_control_demo_description/openduckmini/assets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
- link trunk_assembly: geometry visual mesh filename=package://ros2_control_demo_description/openduckmini/assets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; visual mesh filename=package://ros2_control_demo_description/openduckmini/assets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

File: ros2_control_demo_description/openduckmini/ros2_control/open_duck_mini.ros2_control.xacro (robot description, xacro)
@@ -10,8 +10,8 @@
         <hardware>
           <plugin>ros2_control_demo_example_18/DuckMiniMujocoSystemInterface</plugin>
-          <param name="mujoco_model">$(find ros2_control_demo_example_18)/description/mujoco/scene.xml</param>
-          <param name="meshdir">$(find ros2_control_demo_example_18)/description/assets</param>
+          <param name="mujoco_model">$(find ros2_control_demo_description)/openduckmini/mujoco/scene.xml</param>
+          <param name="meshdir">$(find ros2_control_demo_description)/openduckmini/assets</param>
           <!-- External PID disabled: MuJoCo built-in actuators used -->
-          <param name="override_start_position_file">$(find ros2_control_demo_example_18)/description/mujoco/start_positions.xml</param>
+          <param name="override_start_position_file">$(find ros2_control_demo_description)/openduckmini/mujoco/start_positions.xml</param>
           <param name="headless">${headless}</param>
         </hardware>

File: ros2_control_demo_description/openduckmini/urdf/open_duck_mini.urdf.xacro (robot description, xacro)
@@ -12,7 +12,7 @@
   <!-- Include the base URDF description -->
   <!-- Note: xacro will process the URDF file and merge its content -->
-  <xacro:include filename="$(find ros2_control_demo_example_18)/description/mujoco/robot.urdf" />
+  <xacro:include filename="$(find ros2_control_demo_description)/openduckmini/mujoco/robot.urdf" />
   <!-- Import Open Duck Mini ros2_control description -->
-  <xacro:include filename="$(find ros2_control_demo_example_18)/description/ros2_control/open_duck_mini.ros2_control.xacro" />
+  <xacro:include filename="$(find ros2_control_demo_description)/openduckmini/ros2_control/open_duck_mini.ros2_control.xacro" />
   <xacro:open_duck_mini_ros2_control
     name="OpenDuckMini" prefix="$(arg prefix)" use_mock_hardware="$(arg use_mock_hardware)" headless="$(arg headless)"/>
