Commit message: Align Open Duck Mini joint limits with MJCF and clip ONNX commands

File: ros2_control_demo_description/openduckmini/mujoco/robot.urdf (robot description, URDF)
Before this commit: robot open-duck-mini, 16 links, 15 joints
Joints:
- joint head_pitch: limit lower=-10.0 upper=10.0 effort=3.23 velocity=10.0 -> lower=-0.7853981633974483 upper=0.7853981633974483 effort=3.23 velocity=10.0
- joint head_roll: limit lower=-10.0 upper=10.0 effort=3.23 velocity=10.0 -> lower=-0.523598775598218 upper=0.5235987755983796 effort=3.23 velocity=10.0
- joint head_yaw: limit lower=-10.0 upper=10.0 effort=3.23 velocity=10.0 -> lower=-2.792526803190927 upper=2.792526803190927 effort=3.23 velocity=10.0
- joint left_ankle: limit lower=-10.0 upper=10.0 effort=3.23 velocity=10.0 -> lower=-1.5707963267948957 upper=1.5707963267948974 effort=3.23 velocity=10.0
- joint left_hip_pitch: limit lower=-10.0 upper=10.0 effort=3.23 velocity=10.0 -> lower=-1.2217304763960306 upper=0.5235987755982988 effort=3.23 velocity=10.0
- joint left_hip_roll: limit lower=-10.0 upper=10.0 effort=3.23 velocity=10.0 -> lower=-0.4363323129985815 upper=0.43633231299858327 effort=3.23 velocity=10.0
- joint left_knee: limit lower=-10.0 upper=10.0 effort=3.23 velocity=10.0 -> lower=-1.5707963267948966 upper=1.5707963267948966 effort=3.23 velocity=10.0
- joint neck_pitch: limit lower=-10.0 upper=10.0 effort=3.23 velocity=10.0 -> lower=-0.3490658503988437 upper=1.1344640137963364 effort=3.23 velocity=10.0
- joint right_ankle: limit lower=-10.0 upper=10.0 effort=3.23 velocity=10.0 -> lower=-1.5707963267948957 upper=1.5707963267948974 effort=3.23 velocity=10.0
- joint right_hip_pitch: limit lower=-10.0 upper=10.0 effort=3.23 velocity=10.0 -> lower=-0.5235987755982988 upper=1.2217304763960306 effort=3.23 velocity=10.0
- joint right_knee: limit lower=-10.0 upper=10.0 effort=3.23 velocity=10.0 -> lower=-1.5707963267948966 upper=1.5707963267948966 effort=3.23 velocity=10.0
